Commit message: adding launch, world,urdf,rviz file

File: insect_description/urdf/insect.urdf.xacro (robot description, xacro)
@@ -24,3 +24,237 @@
 <xacro:property name="r_b_hip_mass" value="1.0"/>
 <!--motors parameters-->
-<!-->
+<!--left_front_motor parameters-->
+<xacro:property name="l_f_motor_mass" value="0.8"/>
+<!--left_back_hip parameters-->
+<xacro:property name="r_b_motor_mass" value="0.8"/>
+<!--right_front_hip parameters-->
+<xacro:property name="r_f_motor_mass" value="1.0"/>
+<!--right_back_hip parameters-->
+<xacro:property name="r_b_motor_mass" value="1.0"/>
+<!--#############################################################################################################################-->
+<link name="world"/>
+<link name='torso_base'>
+  <inertial>
+    <mass value="${torso_mass}"/>
+    <!--origin xyz="0 0 0.2" rpy="0 0 0"/-->
+      <!--origin xyz="-0.536511 0.016494 0.000002" rpy="0 0.000004 -0.000730"/-->
+    <inertia
+      ixx="0.08" ixy="0" ixz="0"
+      iyy="0.08" iyz="0"
+      izz="0.08"
+      />
+    </inertial>
+    <collision name='torso_collision'>
+      <origin xyz="0 0 0" rpy="0 0 0"/>
+      <geometry>
+        <mesh filename="file:///home/veer/catkin_ws/src/insect_description/meshes/torso_v1.dae"/>
+      </geometry>
+    </collision>
+    <visual name="torso_visual">
+      <origin xyz="0 0 0" rpy="0 0 0"/>
+      <geometry>
+        <mesh filename="file:///home/veer/catkin_ws/src/insect_description/meshes/torso_v1.dae"/>
+      </geometry>
+    </visual>
+    <sensor name='my_contact' type='contact'>
+          <contact>
+            <collision>torso_collision</collision>
+          </contact>
+    </sensor>
+  </link>
+  <link name= "l_f_motor">
+    <collision name='l_f_motor_collision'>
+      <origin xyz="0 0 0" rpy="0 -0.5 -1.5"/>
+        <geometry>
+          <mesh filename="file:///home/veer/catkin_ws/src/insect_description/meshes/motor_v1.dae"/>
+        </geometry>
+      </collision>
+      <visual name="l_f_motor_visual">
+        <origin xyz="0 0 0" rpy="0 -0.5 -1.5"/>
+        <geometry>
+          <mesh filename="file:///home/veer/catkin_ws/src/insect_description/meshes/motor_v1.dae"/>
+        </geometry>
+      </visual>
+    </link>
+    <link name= "r_f_motor">
+      <collision name='l_f_motor_collision'>
+        <origin xyz="0 0 0" rpy="0 -0.5 1.5"/>
+          <geometry>
+            <mesh filename="file:///home/veer/catkin_ws/src/insect_description/meshes/motor_v1.dae"/>
+          </geometry>
+        </collision>
+        <visual name="r_f_motor_visual">
+          <origin xyz="0 0 0" rpy="0 -0.5 1.5"/>
+          <geometry>
+            <mesh filename="file:///home/veer/catkin_ws/src/insect_description/meshes/motor_v1.dae"/>
+          </geometry>
+        </visual>
+      </link>
+      <link name= "l_b_motor">
+        <collision name='l_b_motor_collision'>
+          <origin xyz="0 0 0" rpy="0 -0.5 -1.5"/>
+            <geometry>
+              <mesh filename="file:///home/veer/catkin_ws/src/insect_description/meshes/motor_v1.dae"/>
+            </geometry>
+          </collision>
+          <visual name="l_b_motor_visual">
+            <origin xyz="0 0 0" rpy="0 -0.5 -1.5"/>
+            <geometry>
+              <mesh filename="file:///home/veer/catkin_ws/src/insect_description/meshes/motor_v1.dae"/>
+            </geometry>
+          </visual>
+        </link>
+        <link name= "r_b_motor">
+          <collision name='r_b_motor_collision'>
+            <origin xyz="0 0 0" rpy="0 -0.5 1.5"/>
+              <geometry>
+                <mesh filename="file:///home/veer/catkin_ws/src/insect_description/meshes/motor_v1.dae"/>
+              </geometry>
+            </collision>
+            <visual name="r_b_motor_visual">
+              <origin xyz="0 0 0" rpy="0 -0.5 1.5"/>
+              <geometry>
+                <mesh filename="file:///home/veer/catkin_ws/src/insect_description/meshes/motor_v1.dae"/>
+              </geometry>
+            </visual>
+          </link>
+          <link name= "l_f_hip">
+            <collision name='l_f_hip_collision'>
+              <origin xyz="0 0 0" rpy="0 -0.5 -1.5"/>
+                <geometry>
+                  <mesh filename="file:///home/veer/catkin_ws/src/insect_description/meshes/hip_v1.dae"/>
+                </geometry>
+              </collision>
+              <visual name="l_f_hip_visual">
+                <origin xyz="0 0 0" rpy="0 -0.5 -1.5"/>
+                <geometry>
+                  <mesh filename="file:///home/veer/catkin_ws/src/insect_description/meshes/hip_v1.dae"/>
+                </geometry>
+              </visual>
+            </link>
+            <link name= "r_f_hip">
+              <collision name='l_f_hip_collision'>
+                <origin xyz="0 0 0" rpy="0 -0.5 1.5"/>
+                  <geometry>
+                    <mesh filename="file:///home/veer/catkin_ws/src/insect_description/meshes/hip_v1.dae"/>
+                  </geometry>
+                </collision>
+                <visual name="r_f_hip_visual">
+                  <origin xyz="0 0 0" rpy="0 -0.5 1.5"/>
+                  <geometry>
+                    <mesh filename="file:///home/veer/catkin_ws/src/insect_description/meshes/hip_v1.dae"/>
+                  </geometry>
+                </visual>
+              </link>
+              <link name= "l_b_hip">
+                <collision name='l_b_hip_collision'>
+                  <origin xyz="0 0 0" rpy="0 -0.5 -1.5"/>
+                    <geometry>
+                      <mesh filename="file:///home/veer/catkin_ws/src/insect_description/meshes/hip_v1.dae"/>
+                    </geometry>
+                  </collision>
+                  <visual name="l_b_hip_visual">
+                    <origin xyz="0 0 0" rpy="0 -0.5 -1.5"/>
+                    <geometry>
+                      <mesh filename="file:///home/veer/catkin_ws/src/insect_description/meshes/hip_v1.dae"/>
+                    </geometry>
+                  </visual>
+                </link>
+                <link name= "r_b_hip">
+                  <collision name='r_b_hip_collision'>
+                    <origin xyz="0 0 0" rpy="0 -0.5 1.5"/>
+                      <geometry>
+                        <mesh filename="file:///home/veer/catkin_ws/src/insect_description/meshes/hip_v1.dae"/>
+                      </geometry>
+                    </collision>
+                    <visual name="r_b_hip_visual">
+                      <origin xyz="0 0 0" rpy="0 -0.5 1.5"/>
+                      <geometry>
+                        <mesh filename="file:///home/veer/catkin_ws/src/insect_description/meshes/hip_v1.dae"/>
+                      </geometry>
+                    </visual>
+                  </link>
+                  <link name= "l_f_h_motor">
+                    <collision name='l_f_h_motor_collision'>
+                      <origin xyz="0 0 0" rpy="0 -3.4 -1.5"/>
+                        <geometry>
+                          <mesh filename="file:///home/veer/catkin_ws/src/insect_description/meshes/motor_h_v1.dae"/>
+                        </geometry>
+                      </collision>
+                      <visual name="l_f_h_motor_visual">
+                        <origin xyz="0 0 0" rpy="0 -3.4 -1.5"/>
+                        <geometry>
+                          <mesh filename="file:///home/veer/catkin_ws/src/insect_description/meshes/motor_h_v1.dae"/>
+                        </geometry>
+                      </visual>
+                    </link>
+                    <link name= "r_f_h_motor">
+                      <collision name='l_f_h_motor_collision'>
+                        <origin xyz="0 0 0" rpy="0 -3.4 -1.5"/>
+                          <geometry>
+                            <mesh filename="file:///home/veer/catkin_ws/src/insect_description/meshes/motor_h_v1.dae"/>
+                          </geometry>
+                        </collision>
+                        <visual name="r_f_h_motor_visual">
+                          <origin xyz="0 0 0" rpy="0 -3.4 1.5"/>
+                          <geometry>
+                            <mesh filename="file:///home/veer/catkin_ws/src/insect_description/meshes/motor_h_v1.dae"/>
+                          </geometry>
+                        </visual>
+                      </link>
+  <joint name="world_joint"  type="fixed">
+    <origin xyz="0 0 0.2" rpy="0 0 0" />
+    <parent link="world"/>
+    <child link="torso_base"/>
+</joint>
+<joint name="l_f_motor_joint"  type="fixed">
+  <origin xyz="0.048 0.08 -0.08" rpy="0 0 0" />
+  <parent link="torso_base"/>
+  <child link="l_f_motor"/>
+</joint>
+<joint name="r_f_motor_joint"  type="fixed">
+  <origin xyz="0.048 -0.09 -0.08" rpy="0 0 0" />
+  <parent link="torso_base"/>
+  <child link="r_f_motor"/>
+</joint>
+<joint name="l_b_motor_joint"  type="fixed">
+  <origin xyz="-0.2 0.08 -0.08" rpy="0 0 0" />
+  <parent link="torso_base"/>
+  <child link="l_b_motor"/>
+</joint>
+<joint name="r_b_motor_joint"  type="fixed">
+  <origin xyz="-0.2 -0.09 -0.08" rpy="0 0 0" />
+  <parent link="torso_base"/>
+  <child link="r_b_motor"/>
+</joint>
+<joint name="l_f_hip_joint"  type="fixed">
+  <origin xyz="0.006 0.01 -0.067" rpy="0 0 0" />
+  <parent link="l_f_motor"/>
+  <child link="l_f_hip"/>
+</joint>
+<joint name="r_f_hip_joint"  type="fixed">
+  <origin xyz="0.006 -0.01 -0.067" rpy="0 0 0" />
+  <parent link="r_f_motor"/>
+  <child link="r_f_hip"/>
+</joint>
+<joint name="l_b_hip_joint"  type="fixed">
+  <origin xyz="0.006 0.01 -0.067" rpy="0 0 0" />
+  <parent link="l_b_motor"/>
+  <child link="l_b_hip"/>
+</joint>
+<joint name="r_b_hip_joint"  type="fixed">
+  <origin xyz="-0.006 -0.01 -0.067" rpy="0 0 0" />
+  <parent link="r_b_motor"/>
+  <child link="r_b_hip"/>
+</joint>
+<joint name="l_f_h_motor_joint"  type="fixed">
+  <origin xyz="-0.013 0.163 0.088" rpy="0 0 0" />
+  <parent link="l_f_hip"/>
+  <child link="l_f_h_motor"/>
+</joint>
+<joint name="r_f_h_motor_joint"  type="fixed">
+  <origin xyz="0.02 -0.155 0.088" rpy="0 0 0" />
+  <parent link="r_f_hip"/>
+  <child link="r_f_h_motor"/>
+</joint>
+</robot>

Commit message: modification of xacro

File: insect_description/urdf/insect.urdf.xacro (robot description, xacro)
@@ -37,5 +37,5 @@
   <inertial>
     <mass value="${torso_mass}"/>
-    <!--origin xyz="0 0 0.2" rpy="0 0 0"/-->
+    <!--origin xyz="0 0 1.0" rpy="0 0 0"/-->
       <!--origin xyz="-0.536511 0.016494 0.000002" rpy="0 0.000004 -0.000730"/-->
     <inertia
@@ -190,5 +190,5 @@
                     </link>
                     <link name= "r_f_h_motor">
-                      <collision name='l_f_h_motor_collision'>
+                      <collision name='r_f_h_motor_collision'>
                         <origin xyz="0 0 0" rpy="0 -3.4 -1.5"/>
                           <geometry>
@@ -203,4 +203,88 @@
                         </visual>
                       </link>
+                      <link name= "l_b_h_motor">
+                        <collision name='l_b_h_motor_collision'>
+                          <origin xyz="0 0 0" rpy="0 -3.4 -1.5"/>
+                            <geometry>
+                              <mesh filename="file:///home/veer/catkin_ws/src/insect_description/meshes/motor_h_v1.dae"/>
+                            </geometry>
+                          </collision>
+                          <visual name="l_b_h_motor_visual">
+                            <origin xyz="0 0 0" rpy="0 -3.4 -1.5"/>
+                            <geometry>
+                              <mesh filename="file:///home/veer/catkin_ws/src/insect_description/meshes/motor_h_v1.dae"/>
+                            </geometry>
+                          </visual>
+                        </link>
+                        <link name= "r_b_h_motor">
+                          <collision name='r_b_h_motor_collision'>
+                            <origin xyz="0 0 0" rpy="0 -3.4 -1.5"/>
+                              <geometry>
+                                <mesh filename="file:///home/veer/catkin_ws/src/insect_description/meshes/motor_h_v1.dae"/>
+                              </geometry>
+                            </collision>
+                            <visual name="r_b_h_motor_visual">
+                              <origin xyz="0 0 0" rpy="0 -3.4 1.5"/>
+                              <geometry>
+                                <mesh filename="file:///home/veer/catkin_ws/src/insect_description/meshes/motor_h_v1.dae"/>
+                              </geometry>
+                            </visual>
+                          </link>
+                          <link name= "l_f_leg">
+                            <collision name='l_f_leg_collision'>
+                              <origin xyz="0 0 0" rpy="0 0 -1.5"/>
+                                <geometry>
+                                  <mesh filename="file:///home/veer/catkin_ws/src/insect_description/meshes/leg_v1.dae"/>
+                                </geometry>
+                              </collision>
+                              <visual name="l_f_legb_visual">
+                                <origin xyz="0 0 0" rpy="0 0 -1.5"/>
+                                <geometry>
+                                  <mesh filename="file:///home/veer/catkin_ws/src/insect_description/meshes/leg_v1.dae"/>
+                                </geometry>
+                              </visual>
+                            </link>
+                            <link name= "l_b_leg">
+                              <collision name='l_b_leg_collision'>
+                                <origin xyz="0 0 0" rpy="0 0 -1.5"/>
+                                  <geometry>
+                                    <mesh filename="file:///home/veer/catkin_ws/src/insect_description/meshes/leg_v1.dae"/>
+                                  </geometry>
+                                </collision>
+                                <visual name="l_b_leg_visual">
+                                  <origin xyz="0 0 0" rpy="0 0 -1.5"/>
+                                  <geometry>
+                                    <mesh filename="file:///home/veer/catkin_ws/src/insect_description/meshes/leg_v1.dae"/>
+                                  </geometry>
+                                </visual>
+                              </link>
+                              <link name= "r_f_leg">
+                                <collision name='r_f_leg_collision'>
+                                  <origin xyz="0 0 0" rpy="0 0 1.5"/>
+                                    <geometry>
+                                      <mesh filename="file:///home/veer/catkin_ws/src/insect_description/meshes/leg_v1.dae"/>
+                                    </geometry>
+                                  </collision>
+                                  <visual name="_f_legb_visual">
+                                    <origin xyz="0 0 0" rpy="0 0 1.5"/>
+                                    <geometry>
+                                      <mesh filename="file:///home/veer/catkin_ws/src/insect_description/meshes/leg_v1.dae"/>
+                                    </geometry>
+                                  </visual>
+                                </link>
+                                <link name= "r_b_leg">
+                                  <collision name='r_b_leg_collision'>
+                                    <origin xyz="0 0 0" rpy="0 0 1.5"/>
+                                      <geometry>
+                                        <mesh filename="file:///home/veer/catkin_ws/src/insect_description/meshes/leg_v1.dae"/>
+                                      </geometry>
+                                    </collision>
+                                    <visual name="r_b_leg_visual">
+                                      <origin xyz="0 0 0" rpy="0 0 1.5"/>
+                                      <geometry>
+                                        <mesh filename="file:///home/veer/catkin_ws/src/insect_description/meshes/leg_v1.dae"/>
+                                      </geometry>
+                                    </visual>
+                                  </link>
   <joint name="world_joint"  type="fixed">
     <origin xyz="0 0 0.2" rpy="0 0 0" />
@@ -249,12 +333,42 @@
 </joint>
 <joint name="l_f_h_motor_joint"  type="fixed">
-  <origin xyz="-0.013 0.163 0.088" rpy="0 0 0" />
+  <origin xyz="-0.014 0.163 0.088" rpy="0 0 0" />
   <parent link="l_f_hip"/>
   <child link="l_f_h_motor"/>
 </joint>
 <joint name="r_f_h_motor_joint"  type="fixed">
-  <origin xyz="0.02 -0.155 0.088" rpy="0 0 0" />
+  <origin xyz="-0.010 -0.165 0.088" rpy="0 0 0" />
   <parent link="r_f_hip"/>
   <child link="r_f_h_motor"/>
 </joint>
+<joint name="l_b_h_motor_joint"  type="fixed">
+  <origin xyz="-0.016 0.165 0.088" rpy="0 0 0" />
+  <parent link="l_b_hip"/>
+  <child link="l_b_h_motor"/>
+</joint>
+<joint name="r_b_h_motor_joint"  type="fixed">
+  <origin xyz="-0.010 -0.165 0.088" rpy="0 0 0" />
+  <parent link="r_b_hip"/>
+  <child link="r_b_h_motor"/>
+</joint>
+<joint name="l_f_leg_joint"  type="fixed">
+  <origin xyz="-0.006 0.07 -0.077" rpy="0 0 0" />
+  <parent link="l_f_h_motor"/>
+  <child link="l_f_leg"/>
+</joint>
+<joint name="l_b_leg_joint"  type="fixed">
+  <origin xyz="-0.006 0.07 -0.077" rpy="0 0 0" />
+  <parent link="l_b_h_motor"/>
+  <child link="l_b_leg"/>
+</joint>
+<joint name="r_f_leg_joint"  type="fixed">
+  <origin xyz="-0.006 -0.07 -0.077" rpy="0 0 0" />
+  <parent link="r_f_h_motor"/>
+  <child link="r_f_leg"/>
+</joint>
+<joint name="r_b_leg_joint"  type="fixed">
+  <origin xyz="-0.006 -0.07 -0.077" rpy="0 0 0" />
+  <parent link="r_b_h_motor"/>
+  <child link="r_b_leg"/>
+</joint>
 </robot>

Commit message: adding servo motor.yaml anf sensor plugin

File: insect_description/urdf/insect.urdf.xacro (robot description, xacro)
@@ -37,5 +37,5 @@
   <inertial>
     <mass value="${torso_mass}"/>
-    <!--origin xyz="0 0 1.0" rpy="0 0 0"/-->
+    <!--origin xyz="0 0 2" rpy="0 0 0"/-->
       <!--origin xyz="-0.536511 0.016494 0.000002" rpy="0 0.000004 -0.000730"/-->
     <inertia
@@ -57,10 +57,25 @@
       </geometry>
     </visual>
-    <sensor name='my_contact' type='contact'>
-          <contact>
-            <collision>torso_collision</collision>
-          </contact>
-    </sensor>
   </link>
+ <!--IMU sensor_link-->
+  <link name="imu_link">
+  <inertial>
+    <mass value="0.001"/>
+    <origin rpy="0 0 0" xyz="0 0 0"/>
+    <inertia ixx="0.0001" ixy="0" ixz="0" iyy="0.000001" iyz="0" izz="0.0001"/>
+  </inertial>
+  <visual>
+    <origin rpy="0 0 0" xyz="0 0 0"/>
+    <geometry>
+      <box size="0.001 0.001 0.001"/> <!--box size="0.001 0.001 0.001"/-->
+    </geometry>
+  </visual>
+  <collision>
+    <origin rpy="0 0 0" xyz="0 0 0"/>
+    <geometry>
+      <box size="0.001 0.001 0.001"/> <!--<box size=".001 .001 .001"/-->
+    </geometry>
+  </collision>
+</link>
   <link name= "l_f_motor">
     <collision name='l_f_motor_collision'>
@@ -372,3 +387,92 @@
   <child link="r_b_leg"/>
 </joint>
+<!--IMU sensor joint-->
+<joint name="imu_joint" type="fixed">
+  <axis xyz="0.01 0 0.01"/> <!-- 0 1 0 -->
+  <origin xyz="0 0 0.05"/>
+  <parent link="torso_base"/>
+  <child link="imu_link"/>
+</joint>
+<!--contact_sensor_torso_base-->
+<gazebo reference="torso_base">
+  <sensor name="contact_sensor" type="contact">
+    <always_on>true</always_on>
+    <updateRate>15.0</updateRate>
+    <contact>
+      <collision>torso_collision</collision>
+    </contact>
+    <plugin filename="libgazebo_ros_bumper.so" name="gazebo_ros_bumper_controller">
+      <bumperTopicName>torso_contact_info</bumperTopicName>
+      <frameName>torso</frameName>
+    </plugin>
+  </sensor>
+</gazebo>
+<!--front_left_leg_contact contact_sensor-->
+<gazebo reference="l_f_leg">
+  <sensor name="contact_sensor_1" type="contact">
+    <always_on>true</always_on>
+    <updateRate>15.0</updateRate>
+    <contact>
+      <collision>l_f_leg_collision</collision>
+    </contact>
+    <plugin filename="libgazebo_ros_bumper.so" name="gazebo_ros_bumper_controller">
+      <bumperTopicName>l_f_leg_contact_info</bumperTopicName>
+      <frameName>l_f_leg</frameName>
+    </plugin>
+  </sensor>
+</gazebo>
+<!--back_left_leg_contact contact_sensor-->
+<gazebo reference="l_b_leg">
+  <sensor name="contact_sensor_2" type="contact">
+    <always_on>true</always_on>
+    <updateRate>15.0</updateRate>
+    <contact>
+      <collision>l_b_leg_collision</collision>
+    </contact>
+    <plugin filename="libgazebo_ros_bumper.so" name="gazebo_ros_bumper_controller">
+      <bumperTopicName>l_b_leg_contact_info</bumperTopicName>
+      <frameName>l_b_leg</frameName>
+    </plugin>
+  </sensor>
+</gazebo>
+<!--frot right_leg_contact contact_sensor-->
+<gazebo reference="r_f_leg">
+  <sensor name="contact_sensor_3" type="contact">
+    <always_on>true</always_on>
+    <updateRate>15.0</updateRate>
+    <contact>
+      <collision>r_f_leg_collision</collision>
+    </contact>
+    <plugin filename="libgazebo_ros_bumper.so" name="gazebo_ros_bumper_controller">
+      <bumperTopicName>r_f_leg_contact_info</bumperTopicName>
+      <frameName>r_f_leg</frameName>
+    </plugin>
+  </sensor>
+</gazebo>
+<!--back right_leg_contact contact_sensor-->
+<gazebo reference="r_b_leg">
+  <sensor name="contact_sensor_4" type="contact">
+    <always_on>true</always_on>
+    <updateRate>15.0</updateRate>
+    <contact>
+      <collision>r_b_leg_collision</collision>
+    </contact>
+    <plugin filename="libgazebo_ros_bumper.so" name="gazebo_ros_bumper_controller">
+      <bumperTopicName>r_b_leg_contact_info</bumperTopicName>
+      <frameName>r_b_leg</frameName>
+    </plugin>
+  </sensor>
+</gazebo>
+<!--plugin for IMU sensor--><!--improve plugin-->
+<gazebo>
+  <plugin name="imu_controller" filename="libgazebo_ros_imu.so">
+    <alwaysOn>true</alwaysOn>
+    <updateRate>50.0</updateRate>
+    <bodyName>imu_link</bodyName>
+    <topicName>imu_data</topicName>
+    <gaussianNoise>2.89e-08</gaussianNoise>
+    <xyzOffsets>0 0 0</xyzOffsets>
+    <rpyOffsets>0 0 0</rpyOffsets>
+  </plugin>
+</gazebo>
 </robot>
