Commit message: modification in xacro

File: insect_description/urdf/insect.urdf.xacro (robot description, xacro)
@@ -3,81 +3,46 @@
 <!--##################################################################################################################################-->
 <!--xacro parameters-->
-<!--torso parameters-->
-<xacro:property name="torso_mass" value="8.0"/>
-<!--legs parameters-->
-<!--left_front_leg parameters-->
-<xacro:property name="l_f_leg_mass" value="0.8"/>
-<!--left_back_leg parameters-->
-<xacro:property name="r_b_leg_mass" value="0.8"/>
-<!--right_front_leg parameters-->
-<xacro:property name="r_f_leg_mass" value="1.0"/>
-<!--right_back_leg parameters-->
-<xacro:property name="r_b_leg_mass" value="1.0"/>
-<!--hips parameters-->
-<!--left_front_hip parameters-->
-<xacro:property name="l_f_hip_mass" value="0.8"/>
-<!--left_back_hip parameters-->
-<xacro:property name="r_b_hip_mass" value="0.8"/>
-<!--right_front_hip parameters-->
-<xacro:property name="r_f_hip_mass" value="1.0"/>
-<!--right_back_hip parameters-->
-<xacro:property name="r_b_hip_mass" value="1.0"/>
-<!--motors parameters-->
-<!--left_front_motor parameters-->
-<xacro:property name="l_f_motor_mass" value="0.8"/>
-<!--left_back_hip parameters-->
-<xacro:property name="r_b_motor_mass" value="0.8"/>
-<!--right_front_hip parameters-->
-<xacro:property name="r_f_motor_mass" value="1.0"/>
-<!--right_back_hip parameters-->
-<xacro:property name="r_b_motor_mass" value="1.0"/>
 <!--#############################################################################################################################-->
+<!--macro param-->
+<xacro:macro name="default_inertial" params="mass">
+   <inertial>
+     <mass value="${mass}" />
+     <inertia ixx="1.0" ixy="0.0" ixz="0.0" iyy="1.0" iyz="0.0" izz="1.0" />
+   </inertial>
+ </xacro:macro>
+<!--####################################################################################################################################-->
 <link name="world"/>
-<link name='torso_base'>
-  <inertial>
-    <mass value="${torso_mass}"/>
-    <!--origin xyz="0 0 2" rpy="0 0 0"/-->
-      <!--origin xyz="-0.536511 0.016494 0.000002" rpy="0 0.000004 -0.000730"/-->
-    <inertia
-      ixx="0.08" ixy="0" ixz="0"
-      iyy="0.08" iyz="0"
-      izz="0.08"
-      />
-    </inertial>
-    <collision name='torso_collision'>
-      <origin xyz="0 0 0" rpy="0 0 0"/>
+<link name="torso_base">
+<collision name="collision">
+  <origin xyz="0 0 0" rpy="0 0 0"/>
+  <geometry>
+    <mesh filename="file:///home/veer/catkin_ws/src/insect_description/meshes/torso_v1.dae"/>
+  </geometry>
+</collision>
+<visual name="visual">
+  <origin xyz="0 0 0" rpy="0 0 0"/>
+  <geometry>
+    <mesh filename="file:///home/veer/catkin_ws/src/insect_description/meshes/torso_v1.dae"/>
+  </geometry>
+</visual>
+<xacro:default_inertial mass="0.8"/>
+</link>
+ <!--IMU sensor_link-->
+  <link name="imu_link">
+    <visual>
+      <origin rpy="0 0 0" xyz="0 0 0"/>
       <geometry>
-        <mesh filename="file:///home/veer/catkin_ws/src/insect_description/meshes/torso_v1.dae"/>
+        <box size="0.001 0.001 0.001"/> <!--box size="0.001 0.001 0.001"/-->
+      </geometry>
+    </visual>
+    <collision>
+      <origin rpy="0 0 0" xyz="0 0 0"/>
+      <geometry>
+        <box size="0.001 0.001 0.001"/> <!--<box size=".001 .001 .001"/-->
       </geometry>
     </collision>
-    <visual name="torso_visual">
-      <origin xyz="0 0 0" rpy="0 0 0"/>
-      <geometry>
-        <mesh filename="file:///home/veer/catkin_ws/src/insect_description/meshes/torso_v1.dae"/>
-      </geometry>
-    </visual>
   </link>
- <!--IMU sensor_link-->
-  <link name="imu_link">
-  <inertial>
-    <mass value="0.001"/>
-    <origin rpy="0 0 0" xyz="0 0 0"/>
-    <inertia ixx="0.0001" ixy="0" ixz="0" iyy="0.000001" iyz="0" izz="0.0001"/>
-  </inertial>
-  <visual>
-    <origin rpy="0 0 0" xyz="0 0 0"/>
-    <geometry>
-      <box size="0.001 0.001 0.001"/> <!--box size="0.001 0.001 0.001"/-->
-    </geometry>
-  </visual>
-  <collision>
-    <origin rpy="0 0 0" xyz="0 0 0"/>
-    <geometry>
-      <box size="0.001 0.001 0.001"/> <!--<box size=".001 .001 .001"/-->
-    </geometry>
-  </collision>
-</link>
   <link name= "l_f_motor">
-    <collision name='l_f_motor_collision'>
+    <collision name="collision">
       <origin xyz="0 0 0" rpy="0 -0.5 -1.5"/>
         <geometry>
@@ -85,13 +50,14 @@
         </geometry>
       </collision>
-      <visual name="l_f_motor_visual">
-        <origin xyz="0 0 0" rpy="0 -0.5 -1.5"/>
+      <visual name="visual">
+        <origin xyz="0 0 0" rpy="0 -0.5 -1.4"/>
         <geometry>
           <mesh filename="file:///home/veer/catkin_ws/src/insect_description/meshes/motor_v1.dae"/>
         </geometry>
       </visual>
+      <xacro:default_inertial mass="0.2"/>
     </link>
     <link name= "r_f_motor">
-      <collision name='l_f_motor_collision'>
+      <collision name="collision">
         <origin xyz="0 0 0" rpy="0 -0.5 1.5"/>
           <geometry>
@@ -99,5 +65,5 @@
           </geometry>
         </collision>
-        <visual name="r_f_motor_visual">
+        <visual name="visual">
           <origin xyz="0 0 0" rpy="0 -0.5 1.5"/>
           <geometry>
@@ -105,7 +71,8 @@
           </geometry>
         </visual>
+        <xacro:default_inertial mass="0.2"/>
       </link>
       <link name= "l_b_motor">
-        <collision name='l_b_motor_collision'>
+        <collision name="collision">
           <origin xyz="0 0 0" rpy="0 -0.5 -1.5"/>
             <geometry>
@@ -113,5 +80,5 @@
             </geometry>
           </collision>
-          <visual name="l_b_motor_visual">
+          <visual name="visual">
             <origin xyz="0 0 0" rpy="0 -0.5 -1.5"/>
             <geometry>
@@ -119,7 +86,8 @@
             </geometry>
           </visual>
+          <xacro:default_inertial mass="0.2"/>
         </link>
         <link name= "r_b_motor">
-          <collision name='r_b_motor_collision'>
+          <collision name="collision">
             <origin xyz="0 0 0" rpy="0 -0.5 1.5"/>
               <geometry>
@@ -127,5 +95,5 @@
               </geometry>
             </collision>
-            <visual name="r_b_motor_visual">
+            <visual name="visual">
               <origin xyz="0 0 0" rpy="0 -0.5 1.5"/>
               <geometry>
@@ -133,7 +101,8 @@
               </geometry>
             </visual>
+            <xacro:default_inertial mass="0.2"/>
           </link>
           <link name= "l_f_hip">
-            <collision name='l_f_hip_collision'>
+            <collision name="collision">
               <origin xyz="0 0 0" rpy="0 -0.5 -1.5"/>
                 <geometry>
@@ -141,5 +110,5 @@
                 </geometry>
               </collision>
-              <visual name="l_f_hip_visual">
+              <visual name="visual">
                 <origin xyz="0 0 0" rpy="0 -0.5 -1.5"/>
                 <geometry>
@@ -147,7 +116,8 @@
                 </geometry>
               </visual>
+              <xacro:default_inertial mass="0.4"/>
             </link>
             <link name= "r_f_hip">
-              <collision name='l_f_hip_collision'>
+              <collision name="collision">
                 <origin xyz="0 0 0" rpy="0 -0.5 1.5"/>
                   <geometry>
@@ -155,5 +125,5 @@
                   </geometry>
                 </collision>
-                <visual name="r_f_hip_visual">
+                <visual name="visual">
                   <origin xyz="0 0 0" rpy="0 -0.5 1.5"/>
                   <geometry>
@@ -161,7 +131,8 @@
                   </geometry>
                 </visual>
+                <xacro:default_inertial mass="0.4"/>
               </link>
               <link name= "l_b_hip">
-                <collision name='l_b_hip_collision'>
+                <collision name="collision">
                   <origin xyz="0 0 0" rpy="0 -0.5 -1.5"/>
                     <geometry>
@@ -169,5 +140,5 @@
                     </geometry>
                   </collision>
-                  <visual name="l_b_hip_visual">
+                  <visual name="visual">
                     <origin xyz="0 0 0" rpy="0 -0.5 -1.5"/>
                     <geometry>
@@ -175,7 +146,8 @@
                     </geometry>
                   </visual>
+                  <xacro:default_inertial mass="0.4"/>
                 </link>
                 <link name= "r_b_hip">
-                  <collision name='r_b_hip_collision'>
+                  <collision name="collision">
                     <origin xyz="0 0 0" rpy="0 -0.5 1.5"/>
                       <geometry>
@@ -183,5 +155,5 @@
                       </geometry>
                     </collision>
-                    <visual name="r_b_hip_visual">
+                    <visual name="visual">
                       <origin xyz="0 0 0" rpy="0 -0.5 1.5"/>
                       <geometry>
@@ -189,7 +161,8 @@
                       </geometry>
                     </visual>
+                    <xacro:default_inertial mass="0.4"/>
                   </link>
                   <link name= "l_f_h_motor">
-                    <collision name='l_f_h_motor_collision'>
+                    <collision name="collision">
                       <origin xyz="0 0 0" rpy="0 -3.4 -1.5"/>
                         <geometry>
@@ -197,5 +170,5 @@
                         </geometry>
                       </collision>
-                      <visual name="l_f_h_motor_visual">
+                      <visual name="visual">
                         <origin xyz="0 0 0" rpy="0 -3.4 -1.5"/>
                         <geometry>
@@ -203,7 +176,8 @@
                         </geometry>
                       </visual>
+                      <xacro:default_inertial mass="0.2"/>
                     </link>
                     <link name= "r_f_h_motor">
-                      <collision name='r_f_h_motor_collision'>
+                      <collision name="collision">
                         <origin xyz="0 0 0" rpy="0 -3.4 -1.5"/>
                           <geometry>
@@ -211,5 +185,5 @@
                           </geometry>
                         </collision>
-                        <visual name="r_f_h_motor_visual">
+                        <visual name="visual">
                           <origin xyz="0 0 0" rpy="0 -3.4 1.5"/>
                           <geometry>
@@ -217,7 +191,8 @@
                           </geometry>
                         </visual>
+                        <xacro:default_inertial mass="0.2"/>
                       </link>
                       <link name= "l_b_h_motor">
-                        <collision name='l_b_h_motor_collision'>
+                        <collision name="collision">
                           <origin xyz="0 0 0" rpy="0 -3.4 -1.5"/>
                             <geometry>
@@ -225,5 +200,5 @@
                             </geometry>
                           </collision>
-                          <visual name="l_b_h_motor_visual">
+                          <visual name="visual">
                             <origin xyz="0 0 0" rpy="0 -3.4 -1.5"/>
                             <geometry>
@@ -231,7 +206,8 @@
                             </geometry>
                           </visual>
+                          <xacro:default_inertial mass="0.2"/>
                         </link>
                         <link name= "r_b_h_motor">
-                          <collision name='r_b_h_motor_collision'>
+                          <collision name="collision">
                             <origin xyz="0 0 0" rpy="0 -3.4 -1.5"/>
                               <geometry>
@@ -239,5 +215,5 @@
                               </geometry>
                             </collision>
-                            <visual name="r_b_h_motor_visual">
+                            <visual name="visual">
                               <origin xyz="0 0 0" rpy="0 -3.4 1.5"/>
                               <geometry>
@@ -245,7 +221,8 @@
                               </geometry>
                             </visual>
+                            <xacro:default_inertial mass="0.2"/>
                           </link>
                           <link name= "l_f_leg">
-                            <collision name='l_f_leg_collision'>
+                            <collision name="collision">
                               <origin xyz="0 0 0" rpy="0 0 -1.5"/>
                                 <geometry>
@@ -253,5 +230,5 @@
                                 </geometry>
                               </collision>
-                              <visual name="l_f_legb_visual">
+                              <visual name="visual">
                                 <origin xyz="0 0 0" rpy="0 0 -1.5"/>
                                 <geometry>
@@ -259,7 +236,8 @@
                                 </geometry>
                               </visual>
+                              <xacro:default_inertial mass="0.4"/>
                             </link>
                             <link name= "l_b_leg">
-                              <collision name='l_b_leg_collision'>
+                              <collision name="collision">
                                 <origin xyz="0 0 0" rpy="0 0 -1.5"/>
                                   <geometry>
@@ -267,5 +245,5 @@
                                   </geometry>
                                 </collision>
-                                <visual name="l_b_leg_visual">
+                                <visual name="visual">
                                   <origin xyz="0 0 0" rpy="0 0 -1.5"/>
                                   <geometry>
@@ -273,7 +251,8 @@
                                   </geometry>
                                 </visual>
+                                <xacro:default_inertial mass="0.4"/>
                               </link>
                               <link name= "r_f_leg">
-                                <collision name='r_f_leg_collision'>
+                                <collision name="collision">
                                   <origin xyz="0 0 0" rpy="0 0 1.5"/>
                                     <geometry>
@@ -281,5 +260,5 @@
                                     </geometry>
                                   </collision>
-                                  <visual name="_f_legb_visual">
+                                  <visual name="visual">
                                     <origin xyz="0 0 0" rpy="0 0 1.5"/>
                                     <geometry>
@@ -287,7 +266,8 @@
                                     </geometry>
                                   </visual>
+                                  <xacro:default_inertial mass="0.4"/>
                                 </link>
                                 <link name= "r_b_leg">
-                                  <collision name='r_b_leg_collision'>
+                                  <collision name="collision">
                                     <origin xyz="0 0 0" rpy="0 0 1.5"/>
                                       <geometry>
@@ -295,5 +275,5 @@
                                       </geometry>
                                     </collision>
-                                    <visual name="r_b_leg_visual">
+                                    <visual name="visual">
                                       <origin xyz="0 0 0" rpy="0 0 1.5"/>
                                       <geometry>
@@ -301,89 +281,14 @@
                                       </geometry>
                                     </visual>
+                                    <xacro:default_inertial mass="0.4"/>
                                   </link>
-  <joint name="world_joint"  type="fixed">
-    <origin xyz="0 0 0.2" rpy="0 0 0" />
-    <parent link="world"/>
-    <child link="torso_base"/>
-</joint>
-<joint name="l_f_motor_joint"  type="fixed">
-  <origin xyz="0.048 0.08 -0.08" rpy="0 0 0" />
-  <parent link="torso_base"/>
-  <child link="l_f_motor"/>
-</joint>
-<joint name="r_f_motor_joint"  type="fixed">
-  <origin xyz="0.048 -0.09 -0.08" rpy="0 0 0" />
-  <parent link="torso_base"/>
-  <child link="r_f_motor"/>
-</joint>
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