Commit message: add PID controller

File: insect_description/urdf/insect.urdf.xacro (robot description, xacro)
@@ -17,5 +17,5 @@
   <origin xyz="0 0 0" rpy="0 0 0"/>
   <geometry>
-    <mesh filename="file:///home/veer/catkin_ws/src/insect_description/meshes/torso_v1.dae"/>
+    <mesh filename="file:///home/rit/catkin_ws2/src/insect_robot/insect_description/meshes/torso_v1.dae"/>
   </geometry>
 </collision>
@@ -23,5 +23,5 @@
   <origin xyz="0 0 0" rpy="0 0 0"/>
   <geometry>
-    <mesh filename="file:///home/veer/catkin_ws/src/insect_description/meshes/torso_v1.dae"/>
+    <mesh filename="file:///home/rit/catkin_ws2/src/insect_robot/insect_description/meshes/torso_v1.dae"/>
   </geometry>
 </visual>
@@ -47,5 +47,5 @@
       <origin xyz="0 0 0" rpy="0 -0.5 -1.5"/>
         <geometry>
-          <mesh filename="file:///home/veer/catkin_ws/src/insect_description/meshes/motor_v1.dae"/>
+          <mesh filename="file:///home/rit/catkin_ws2/src/insect_robot/insect_description/meshes/motor_v1.dae"/>
         </geometry>
       </collision>
@@ -53,5 +53,5 @@
         <origin xyz="0 0 0" rpy="0 -0.5 -1.4"/>
         <geometry>
-          <mesh filename="file:///home/veer/catkin_ws/src/insect_description/meshes/motor_v1.dae"/>
+          <mesh filename="file:///home/rit/catkin_ws2/src/insect_robot/insect_description/meshes/motor_v1.dae"/>
         </geometry>
       </visual>
@@ -62,5 +62,5 @@
         <origin xyz="0 0 0" rpy="0 -0.5 1.5"/>
           <geometry>
-            <mesh filename="file:///home/veer/catkin_ws/src/insect_description/meshes/motor_v1.dae"/>
+            <mesh filename="file:///home/rit/catkin_ws2/src/insect_robot/insect_description/meshes/motor_v1.dae"/>
           </geometry>
         </collision>
@@ -68,5 +68,5 @@
           <origin xyz="0 0 0" rpy="0 -0.5 1.5"/>
           <geometry>
-            <mesh filename="file:///home/veer/catkin_ws/src/insect_description/meshes/motor_v1.dae"/>
+            <mesh filename="file:///home/rit/catkin_ws2/src/insect_robot/insect_description/meshes/motor_v1.dae"/>
           </geometry>
         </visual>
@@ -77,5 +77,5 @@
           <origin xyz="0 0 0" rpy="0 -0.5 -1.5"/>
             <geometry>
-              <mesh filename="file:///home/veer/catkin_ws/src/insect_description/meshes/motor_v1.dae"/>
+              <mesh filename="file:///home/rit/catkin_ws2/src/insect_robot/insect_description/meshes/motor_v1.dae"/>
             </geometry>
           </collision>
@@ -83,5 +83,5 @@
             <origin xyz="0 0 0" rpy="0 -0.5 -1.5"/>
             <geometry>
-              <mesh filename="file:///home/veer/catkin_ws/src/insect_description/meshes/motor_v1.dae"/>
+              <mesh filename="file:///home/rit/catkin_ws2/src/insect_robot/insect_description/meshes/motor_v1.dae"/>
             </geometry>
           </visual>
@@ -92,5 +92,5 @@
             <origin xyz="0 0 0" rpy="0 -0.5 1.5"/>
               <geometry>
-                <mesh filename="file:///home/veer/catkin_ws/src/insect_description/meshes/motor_v1.dae"/>
+                <mesh filename="file:///home/rit/catkin_ws2/src/insect_robot/insect_description/meshes/motor_v1.dae"/>
               </geometry>
             </collision>
@@ -98,5 +98,5 @@
               <origin xyz="0 0 0" rpy="0 -0.5 1.5"/>
               <geometry>
-                <mesh filename="file:///home/veer/catkin_ws/src/insect_description/meshes/motor_v1.dae"/>
+                <mesh filename="file:///home/rit/catkin_ws2/src/insect_robot/insect_description/meshes/motor_v1.dae"/>
               </geometry>
             </visual>
@@ -107,5 +107,5 @@
               <origin xyz="0 0 0" rpy="0 -0.5 -1.5"/>
                 <geometry>
-                  <mesh filename="file:///home/veer/catkin_ws/src/insect_description/meshes/hip_v1.dae"/>
+                  <mesh filename="file:///home/rit/catkin_ws2/src/insect_robot/insect_description/meshes/hip_v1.dae"/>
                 </geometry>
               </collision>
@@ -113,5 +113,5 @@
                 <origin xyz="0 0 0" rpy="0 -0.5 -1.5"/>
                 <geometry>
-                  <mesh filename="file:///home/veer/catkin_ws/src/insect_description/meshes/hip_v1.dae"/>
+                  <mesh filename="file:///home/rit/catkin_ws2/src/insect_robot/insect_description/meshes/hip_v1.dae"/>
                 </geometry>
               </visual>
@@ -122,5 +122,5 @@
                 <origin xyz="0 0 0" rpy="0 -0.5 1.5"/>
                   <geometry>
-                    <mesh filename="file:///home/veer/catkin_ws/src/insect_description/meshes/hip_v1.dae"/>
+                    <mesh filename="file:///home/rit/catkin_ws2/src/insect_robot/insect_description/meshes/hip_v1.dae"/>
                   </geometry>
                 </collision>
@@ -128,5 +128,5 @@
                   <origin xyz="0 0 0" rpy="0 -0.5 1.5"/>
                   <geometry>
-                    <mesh filename="file:///home/veer/catkin_ws/src/insect_description/meshes/hip_v1.dae"/>
+                    <mesh filename="file:///home/rit/catkin_ws2/src/insect_robot/insect_description/meshes/hip_v1.dae"/>
                   </geometry>
                 </visual>
@@ -137,5 +137,5 @@
                   <origin xyz="0 0 0" rpy="0 -0.5 -1.5"/>
                     <geometry>
-                      <mesh filename="file:///home/veer/catkin_ws/src/insect_description/meshes/hip_v1.dae"/>
+                      <mesh filename="file:///home/rit/catkin_ws2/src/insect_robot/insect_description/meshes/hip_v1.dae"/>
                     </geometry>
                   </collision>
@@ -143,5 +143,5 @@
                     <origin xyz="0 0 0" rpy="0 -0.5 -1.5"/>
                     <geometry>
-                      <mesh filename="file:///home/veer/catkin_ws/src/insect_description/meshes/hip_v1.dae"/>
+                      <mesh filename="file:///home/rit/catkin_ws2/src/insect_robot/insect_description/meshes/hip_v1.dae"/>
                     </geometry>
                   </visual>
@@ -152,5 +152,5 @@
                     <origin xyz="0 0 0" rpy="0 -0.5 1.5"/>
                       <geometry>
-                        <mesh filename="file:///home/veer/catkin_ws/src/insect_description/meshes/hip_v1.dae"/>
+                        <mesh filename="file:///home/rit/catkin_ws2/src/insect_robot/insect_description/meshes/hip_v1.dae"/>
                       </geometry>
                     </collision>
@@ -158,5 +158,5 @@
                       <origin xyz="0 0 0" rpy="0 -0.5 1.5"/>
                       <geometry>
-                        <mesh filename="file:///home/veer/catkin_ws/src/insect_description/meshes/hip_v1.dae"/>
+                        <mesh filename="file:///home/rit/catkin_ws2/src/insect_robot/insect_description/meshes/hip_v1.dae"/>
                       </geometry>
                     </visual>
@@ -167,5 +167,5 @@
                       <origin xyz="0 0 0" rpy="0 -3.4 -1.5"/>
                         <geometry>
-                          <mesh filename="file:///home/veer/catkin_ws/src/insect_description/meshes/motor_h_v1.dae"/>
+                          <mesh filename="file:///home/rit/catkin_ws2/src/insect_robot/insect_description/meshes/motor_h_v1.dae"/>
                         </geometry>
                       </collision>
@@ -173,5 +173,5 @@
                         <origin xyz="0 0 0" rpy="0 -3.4 -1.5"/>
                         <geometry>
-                          <mesh filename="file:///home/veer/catkin_ws/src/insect_description/meshes/motor_h_v1.dae"/>
+                          <mesh filename="file:///home/rit/catkin_ws2/src/insect_robot/insect_description/meshes/motor_h_v1.dae"/>
                         </geometry>
                       </visual>
@@ -182,5 +182,5 @@
                         <origin xyz="0 0 0" rpy="0 -3.4 -1.5"/>
                           <geometry>
-                            <mesh filename="file:///home/veer/catkin_ws/src/insect_description/meshes/motor_h_v1.dae"/>
+                            <mesh filename="file:///home/rit/catkin_ws2/src/insect_robot/insect_description/meshes/motor_h_v1.dae"/>
                           </geometry>
                         </collision>
@@ -188,5 +188,5 @@
                           <origin xyz="0 0 0" rpy="0 -3.4 1.5"/>
                           <geometry>
-                            <mesh filename="file:///home/veer/catkin_ws/src/insect_description/meshes/motor_h_v1.dae"/>
+                            <mesh filename="file:///home/rit/catkin_ws2/src/insect_robot/insect_description/meshes/motor_h_v1.dae"/>
                           </geometry>
                         </visual>
@@ -197,5 +197,5 @@
                           <origin xyz="0 0 0" rpy="0 -3.4 -1.5"/>
                             <geometry>
-                              <mesh filename="file:///home/veer/catkin_ws/src/insect_description/meshes/motor_h_v1.dae"/>
+                              <mesh filename="file:///home/rit/catkin_ws2/src/insect_robot/insect_description/meshes/motor_h_v1.dae"/>
                             </geometry>
                           </collision>
@@ -203,5 +203,5 @@
                             <origin xyz="0 0 0" rpy="0 -3.4 -1.5"/>
                             <geometry>
-                              <mesh filename="file:///home/veer/catkin_ws/src/insect_description/meshes/motor_h_v1.dae"/>
+                              <mesh filename="file:///home/rit/catkin_ws2/src/insect_robot/insect_description/meshes/motor_h_v1.dae"/>
                             </geometry>
                           </visual>
@@ -212,5 +212,5 @@
                             <origin xyz="0 0 0" rpy="0 -3.4 -1.5"/>
                               <geometry>
-                                <mesh filename="file:///home/veer/catkin_ws/src/insect_description/meshes/motor_h_v1.dae"/>
+                                <mesh filename="file:///home/rit/catkin_ws2/src/insect_robot/insect_description/meshes/motor_h_v1.dae"/>
                               </geometry>
                             </collision>
@@ -218,5 +218,5 @@
                               <origin xyz="0 0 0" rpy="0 -3.4 1.5"/>
                               <geometry>
-                                <mesh filename="file:///home/veer/catkin_ws/src/insect_description/meshes/motor_h_v1.dae"/>
+                                <mesh filename="file:///home/rit/catkin_ws2/src/insect_robot/insect_description/meshes/motor_h_v1.dae"/>
                               </geometry>
                             </visual>
@@ -227,5 +227,5 @@
                               <origin xyz="0 0 0" rpy="0 0 -1.5"/>
                                 <geometry>
-                                  <mesh filename="file:///home/veer/catkin_ws/src/insect_description/meshes/leg_v1.dae"/>
+                                  <mesh filename="file:///home/rit/catkin_ws2/src/insect_robot/insect_description/meshes/leg_v1.dae"/>
                                 </geometry>
                               </collision>
@@ -233,5 +233,5 @@
                                 <origin xyz="0 0 0" rpy="0 0 -1.5"/>
                                 <geometry>
-                                  <mesh filename="file:///home/veer/catkin_ws/src/insect_description/meshes/leg_v1.dae"/>
+                                  <mesh filename="file:///home/rit/catkin_ws2/src/insect_robot/insect_description/meshes/leg_v1.dae"/>
                                 </geometry>
                               </visual>
@@ -242,5 +242,5 @@
                                 <origin xyz="0 0 0" rpy="0 0 -1.5"/>
                                   <geometry>
-                                    <mesh filename="file:///home/veer/catkin_ws/src/insect_description/meshes/leg_v1.dae"/>
+                                    <mesh filename="file:///home/rit/catkin_ws2/src/insect_robot/insect_description/meshes/leg_v1.dae"/>
                                   </geometry>
                                 </collision>
@@ -248,5 +248,5 @@
                                   <origin xyz="0 0 0" rpy="0 0 -1.5"/>
                                   <geometry>
-                                    <mesh filename="file:///home/veer/catkin_ws/src/insect_description/meshes/leg_v1.dae"/>
+                                    <mesh filename="file:///home/rit/catkin_ws2/src/insect_robot/insect_description/meshes/leg_v1.dae"/>
                                   </geometry>
                                 </visual>
@@ -257,5 +257,5 @@
                                   <origin xyz="0 0 0" rpy="0 0 1.5"/>
                                     <geometry>
-                                      <mesh filename="file:///home/veer/catkin_ws/src/insect_description/meshes/leg_v1.dae"/>
+                                      <mesh filename="file:///home/rit/catkin_ws2/src/insect_robot/insect_description/meshes/leg_v1.dae"/>
                                     </geometry>
                                   </collision>
@@ -263,5 +263,5 @@
                                     <origin xyz="0 0 0" rpy="0 0 1.5"/>
                                     <geometry>
-                                      <mesh filename="file:///home/veer/catkin_ws/src/insect_description/meshes/leg_v1.dae"/>
+                                      <mesh filename="file:///home/rit/catkin_ws2/src/insect_robot/insect_description/meshes/leg_v1.dae"/>
                                     </geometry>
                                   </visual>
@@ -272,5 +272,5 @@
                                     <origin xyz="0 0 0" rpy="0 0 1.5"/>
                                       <geometry>
-                                        <mesh filename="file:///home/veer/catkin_ws/src/insect_description/meshes/leg_v1.dae"/>
+                                        <mesh filename="file:///home/rit/catkin_ws2/src/insect_robot/insect_description/meshes/leg_v1.dae"/>
                                       </geometry>
                                     </collision>
@@ -278,5 +278,5 @@
                                       <origin xyz="0 0 0" rpy="0 0 1.5"/>
                                       <geometry>
-                                        <mesh filename="file:///home/veer/catkin_ws/src/insect_description/meshes/leg_v1.dae"/>
+                                        <mesh filename="file:///home/rit/catkin_ws2/src/insect_robot/insect_description/meshes/leg_v1.dae"/>
                                       </geometry>
                                     </visual>
@@ -299,5 +299,5 @@
   <child link="imu_link"/>
 </joint>
-<joint name="l_f_motor_joint"  type="fixed">
+<joint name="l_f_motor_joint"  type="revolute">
   <origin xyz="0.048 0.08 -0.08" rpy="0 0 0" />
   <parent link="torso_base"/>
@@ -307,5 +307,5 @@
   <joint_properties damping="1.0" friction="1.0"/>
 </joint>
-<joint name="r_f_motor_joint"  type="fixed">
+<joint name="r_f_motor_joint"  type="revolute">
   <origin xyz="0.048 -0.09 -0.08" rpy="0 0 0" />
   <parent link="torso_base"/>
@@ -315,5 +315,5 @@
   <joint_properties damping="1.0" friction="1.0"/>
 </joint>
-<joint name="l_b_motor_joint"  type="fixed">
+<joint name="l_b_motor_joint"  type="revolute">
   <origin xyz="-0.2 0.08 -0.08" rpy="0 0 0" />
   <parent link="torso_base"/>
@@ -323,5 +323,5 @@
   <joint_properties damping="1.0" friction="1.0"/>
 </joint>
-<joint name="r_b_motor_joint"  type="fixed">
+<joint name="r_b_motor_joint"  type="revolute">
   <origin xyz="-0.2 -0.09 -0.08" rpy="0 0 0" />
   <parent link="torso_base"/>
@@ -363,5 +363,5 @@
   <joint_properties damping="1.0" friction="1.0"/>
 </joint>
-<joint name="l_f_h_motor_joint"  type="fixed">
+<joint name="l_f_h_motor_joint"  type="revolute">
   <origin xyz="-0.014 0.163 0.088" rpy="0 0 0" />
   <parent link="l_f_hip"/>
@@ -371,5 +371,5 @@
   <joint_properties damping="1.0" friction="1.0"/>
 </joint>
-<joint name="r_f_h_motor_joint"  type="fixed">
+<joint name="r_f_h_motor_joint"  type="revolute">
   <origin xyz="-0.010 -0.165 0.088" rpy="0 0 0" />
   <parent link="r_f_hip"/>
@@ -379,5 +379,5 @@
   <joint_properties damping="1.0" friction="1.0"/>
 </joint>
-<joint name="l_b_h_motor_joint"  type="fixed">
+<joint name="l_b_h_motor_joint"  type="revolute">
   <origin xyz="-0.016 0.165 0.088" rpy="0 0 0" />
   <parent link="l_b_hip"/>
@@ -387,5 +387,5 @@
   <joint_properties damping="1.0" friction="1.0"/>
 </joint>
-<joint name="r_b_h_motor_joint"  type="fixed">
+<joint name="r_b_h_motor_joint"  type="revolute">
   <origin xyz="-0.010 -0.165 0.088" rpy="0 0 0" />
   <parent link="r_b_hip"/>
@@ -428,4 +428,91 @@
 </joint>
 <!--######################################################################################################################################-->
+<transmission name="l_f_motor_transmission">
+ <type>transmission_interface/SimpleTransmission</type>
+ <joint name="l_f_motor_joint">
+   <hardwareInterface>hardware_interface/EffortJointInterface</hardwareInterface>
+ </joint>
+ <actuator name="l_f_motor">
+   <hardwareInterface>hardware_interface/EffortJointInterface</hardwareInterface>
+   <mechanicalReduction>1</mechanicalReduction>
+ </actuator>
+</transmission>
+<transmission name="l_b_motor_transmission">
+  <type>transmission_interface/SimpleTransmission</type>
+  <joint name="l_b_motor_joint">
+    <hardwareInterface>hardware_interface/EffortJointInterface</hardwareInterface>
+  </joint>
+  <actuator name="l_b_motor">
+    <hardwareInterface>hardware_interface/EffortJointInterface</hardwareInterface>
+    <mechanicalReduction>1</mechanicalReduction>
+  </actuator>
+</transmission>
+<transmission name="r_f_motor_tranmission">
+  <type>transmission_interface/SimpleTransmission</type>
+  <joint name="r_f_motor_joint">
+    <hardwareInterface>hardware_interface/EffortJointInterface</hardwareInterface>
+  </joint>
+  <actuator name="r_f_motor">
+    <hardwareInterface>hardware_interface/EffortJointInterface</hardwareInterface>
+    <mechanicalReduction>1</mechanicalReduction>
+  </actuator>
+</transmission>
+<transmission name="r_b_motor_transmission">
+  <type>transmission_interface/SimpleTransmission</type>
+  <joint name="r_b_motor_joint">
+    <hardwareInterface>hardware_interface/EffortJointInterface</hardwareInterface>
+  </joint>
+  <actuator name="r_b_motor">
+    <hardwareInterface>hardware_interface/EffortJointInterface</hardwareInterface>
+    <mechanicalReduction>1</mechanicalReduction>
+  </actuator>
+</transmission>
+<transmission name="l_f_h_motor_transmission">
+  <type>transmission_interface/SimpleTransmission</type>
+  <joint name="l_f_h_motor_joint">
+    <hardwareInterface>hardware_interface/EffortJointInterface</hardwareInterface>
+  </joint>
+  <actuator name="l_f_h_motor">
+    <hardwareInterface>hardware_interface/EffortJointInterface</hardwareInterface>
+    <mechanicalReduction>1</mechanicalReduction>
+  </actuator>
+</transmission>
+<transmission name="l_b_h_motor_transmission">
+   <type>transmission_interface/SimpleTransmission</type>
+   <joint name="l_b_h_motor_joint">
+     <hardwareInterface>hardware_interface/EffortJointInterface</hardwareInterface>
+   </joint>
+   <actuator name="l_b_h_motor">
+     <hardwareInterface>hardware_interface/EffortJointInterface</hardwareInterface>
+     <mechanicalReduction>1</mechanicalReduction>
+   </actuator>
+ </transmission>
+ <transmission name="r_f_h_motor_transmission">
+   <type>transmission_interface/SimpleTransmission</type>
+   <joint name="r_f_h_motor_joint">
+     <hardwareInterface>hardware_interface/EffortJointInterface</hardwareInterface>
+   </joint>
+   <actuator name="r_f_h_motor">
+     <hardwareInterface>hardware_interface/EffortJointInterface</hardwareInterface>
+     <mechanicalReduction>1</mechanicalReduction>
+   </actuator>
+ </transmission>
+ <transmission name="r_b_h_motor_transmission">
+   <type>transmission_interface/SimpleTransmission</type>
+   <joint name="r_b_h_motor_joint">
+     <hardwareInterface>hardware_interface/EffortJointInterface</hardwareInterface>
+   </joint>
+   <actuator name="r_b_h_motor">
+     <hardwareInterface>hardware_interface/EffortJointInterface</hardwareInterface>
+     <mechanicalReduction>1</mechanicalReduction>
+   </actuator>
+ </transmission>
+<!--##################################################################################################################################-->
+<gazebo>
+  <plugin name="gazebo_ros_control" filename="libgazebo_ros_control.so">
+    <robotNamespace>/insect_robot</robotNamespace>
+    <robotSimType>gazebo_ros_control/DefaultRobotHWSim</robotSimType>
+  </plugin>
+</gazebo>
 <!--contact_sensor_torso_base-->
 <gazebo reference="torso_base">
