Commit message: adding controller and navigation planner for robot

File: insect_description/urdf/insect.urdf.xacro (robot description, xacro)
@@ -283,5 +283,41 @@
                                     <xacro:default_inertial mass="0.4"/>
                                   </link>
+<!--############################################################################################################################-->
+                                  <link name="hokuyo_link">
+                                      <collision>
+                                          <origin xyz="0 0 0" rpy="0 0 0"/>
+                                          <geometry>
+                                              <box size="0.1 0.1 0.1"/>
+                                          </geometry>
+                                      </collision>     <origin xyz="0 0 0" rpy="0 0 0"/>
+                                          <geometry>
+                                              <!--mesh filename="package://insect/meshes/hokuyo.dae"/-->
+                                              <mesh filename="file:///home/rit/catkin_ws2/src/insect_robot/insect_description/meshes/hokuyo.dae"/>
+                                          </geometry>
+                                      <visual>
+                                          <origin xyz="0 0 0" rpy="0 0 0"/>
+                                          <geometry>
+                                              <!--mesh filename="package://insect/meshes/hokuyo.dae"/-->
+                                              <mesh filename="file:///home/rit/catkin_ws2/src/insect_robot/insect_description/meshes/hokuyo.dae"/>
+                                          </geometry>
+                                      </visual>
+                                      <inertial>
+                                          <mass value="1e-5" />
+                                          <origin xyz="0 0 0" rpy="0 0 0"/>
+                                          <inertia ixx="1e-6" ixy="0" ixz="0" iyy="1e-6" iyz="0" izz="1e-6" />
+                                      </inertial>
+                                  </link>
 <!--#########################################################################################################################################-->
+<!-- Joint properties -->
+<xacro:property name="joint_lower_limit" value="-${3.14}"/>
+<xacro:property name="joint_upper_limit" value="${3.14}"/>
+<xacro:property name="joint_effort" value="6.0"/>
+<xacro:property name="joint_velocity" value="0.524"/>
+<!--######################################################################################################################################-->
+<joint name="hokuyo_joint" type="fixed">
+    <origin xyz="0.04 0 0.08" rpy="0 0 0"/>
+    <parent link="torso_base"/>
+    <child link="hokuyo_link"/>
+</joint>
 <joint name="world_joint"  type="fixed">
   <origin xyz="0 0 0.30" rpy="0 0 0" />
@@ -299,5 +335,5 @@
   <child link="imu_link"/>
 </joint>
-<joint name="l_f_motor_joint"  type="revolute">
+<joint name="l_f_motor_joint"  type="fixed">
   <origin xyz="0.048 0.08 -0.08" rpy="0 0 0" />
   <parent link="torso_base"/>
@@ -307,5 +343,5 @@
   <joint_properties damping="1.0" friction="1.0"/>
 </joint>
-<joint name="r_f_motor_joint"  type="revolute">
+<joint name="r_f_motor_joint"  type="fixed">
   <origin xyz="0.048 -0.09 -0.08" rpy="0 0 0" />
   <parent link="torso_base"/>
@@ -315,5 +351,5 @@
   <joint_properties damping="1.0" friction="1.0"/>
 </joint>
-<joint name="l_b_motor_joint"  type="revolute">
+<joint name="l_b_motor_joint"  type="fixed">
   <origin xyz="-0.2 0.08 -0.08" rpy="0 0 0" />
   <parent link="torso_base"/>
@@ -323,5 +359,5 @@
   <joint_properties damping="1.0" friction="1.0"/>
 </joint>
-<joint name="r_b_motor_joint"  type="revolute">
+<joint name="r_b_motor_joint"  type="fixed">
   <origin xyz="-0.2 -0.09 -0.08" rpy="0 0 0" />
   <parent link="torso_base"/>
@@ -363,5 +399,5 @@
   <joint_properties damping="1.0" friction="1.0"/>
 </joint>
-<joint name="l_f_h_motor_joint"  type="revolute">
+<joint name="l_f_h_motor_joint"  type="fixed">
   <origin xyz="-0.014 0.163 0.088" rpy="0 0 0" />
   <parent link="l_f_hip"/>
@@ -371,5 +407,5 @@
   <joint_properties damping="1.0" friction="1.0"/>
 </joint>
-<joint name="r_f_h_motor_joint"  type="revolute">
+<joint name="r_f_h_motor_joint"  type="fixed">
   <origin xyz="-0.010 -0.165 0.088" rpy="0 0 0" />
   <parent link="r_f_hip"/>
@@ -379,5 +415,5 @@
   <joint_properties damping="1.0" friction="1.0"/>
 </joint>
-<joint name="l_b_h_motor_joint"  type="revolute">
+<joint name="l_b_h_motor_joint"  type="fixed">
   <origin xyz="-0.016 0.165 0.088" rpy="0 0 0" />
   <parent link="l_b_hip"/>
@@ -387,5 +423,5 @@
   <joint_properties damping="1.0" friction="1.0"/>
 </joint>
-<joint name="r_b_h_motor_joint"  type="revolute">
+<joint name="r_b_h_motor_joint"  type="fixed">
   <origin xyz="-0.010 -0.165 0.088" rpy="0 0 0" />
   <parent link="r_b_hip"/>
@@ -428,91 +464,85 @@
 </joint>
 <!--######################################################################################################################################-->
-<transmission name="l_f_motor_transmission">
- <type>transmission_interface/SimpleTransmission</type>
- <joint name="l_f_motor_joint">
-   <hardwareInterface>hardware_interface/EffortJointInterface</hardwareInterface>
- </joint>
- <actuator name="l_f_motor">
-   <hardwareInterface>hardware_interface/EffortJointInterface</hardwareInterface>
-   <mechanicalReduction>1</mechanicalReduction>
- </actuator>
-</transmission>
-<transmission name="l_b_motor_transmission">
+<!--transmission name="l_f_motor_transmission">
   <type>transmission_interface/SimpleTransmission</type>
-  <joint name="l_b_motor_joint">
-    <hardwareInterface>hardware_interface/EffortJointInterface</hardwareInterface>
+  <joint name="l_f_motor_joint">
+    <hardwareInterface>EffortJointInterface</hardwareInterface>
   </joint>
-  <actuator name="l_b_motor">
-    <hardwareInterface>hardware_interface/EffortJointInterface</hardwareInterface>
+  <actuator name="l_f_m1">
+    <hardwareInterface>EffortJointInterface</hardwareInterface>
     <mechanicalReduction>1</mechanicalReduction>
   </actuator>
 </transmission>
-<transmission name="r_f_motor_tranmission">
-  <type>transmission_interface/SimpleTransmission</type>
-  <joint name="r_f_motor_joint">
-    <hardwareInterface>hardware_interface/EffortJointInterface</hardwareInterface>
-  </joint>
-  <actuator name="r_f_motor">
-    <hardwareInterface>hardware_interface/EffortJointInterface</hardwareInterface>
-    <mechanicalReduction>1</mechanicalReduction>
-  </actuator>
-</transmission>
-<transmission name="r_b_motor_transmission">
-  <type>transmission_interface/SimpleTransmission</type>
-  <joint name="r_b_motor_joint">
-    <hardwareInterface>hardware_interface/EffortJointInterface</hardwareInterface>
-  </joint>
-  <actuator name="r_b_motor">
-    <hardwareInterface>hardware_interface/EffortJointInterface</hardwareInterface>
-    <mechanicalReduction>1</mechanicalReduction>
-  </actuator>
-</transmission>
-<transmission name="l_f_h_motor_transmission">
-  <type>transmission_interface/SimpleTransmission</type>
-  <joint name="l_f_h_motor_joint">
-    <hardwareInterface>hardware_interface/EffortJointInterface</hardwareInterface>
-  </joint>
-  <actuator name="l_f_h_motor">
-    <hardwareInterface>hardware_interface/EffortJointInterface</hardwareInterface>
-    <mechanicalReduction>1</mechanicalReduction>
-  </actuator>
-</transmission>
-<transmission name="l_b_h_motor_transmission">
-   <type>transmission_interface/SimpleTransmission</type>
-   <joint name="l_b_h_motor_joint">
-     <hardwareInterface>hardware_interface/EffortJointInterface</hardwareInterface>
-   </joint>
-   <actuator name="l_b_h_motor">
-     <hardwareInterface>hardware_interface/EffortJointInterface</hardwareInterface>
-     <mechanicalReduction>1</mechanicalReduction>
-   </actuator>
- </transmission>
- <transmission name="r_f_h_motor_transmission">
-   <type>transmission_interface/SimpleTransmission</type>
-   <joint name="r_f_h_motor_joint">
-     <hardwareInterface>hardware_interface/EffortJointInterface</hardwareInterface>
-   </joint>
-   <actuator name="r_f_h_motor">
-     <hardwareInterface>hardware_interface/EffortJointInterface</hardwareInterface>
-     <mechanicalReduction>1</mechanicalReduction>
-   </actuator>
- </transmission>
- <transmission name="r_b_h_motor_transmission">
-   <type>transmission_interface/SimpleTransmission</type>
-   <joint name="r_b_h_motor_joint">
-     <hardwareInterface>hardware_interface/EffortJointInterface</hardwareInterface>
-   </joint>
-   <actuator name="r_b_h_motor">
-     <hardwareInterface>hardware_interface/EffortJointInterface</hardwareInterface>
-     <mechanicalReduction>1</mechanicalReduction>
-   </actuator>
- </transmission>
-<!--##################################################################################################################################-->
-<gazebo>
-  <plugin name="gazebo_ros_control" filename="libgazebo_ros_control.so">
-    <robotNamespace>/insect_robot</robotNamespace>
-    <robotSimType>gazebo_ros_control/DefaultRobotHWSim</robotSimType>
-  </plugin>
-</gazebo>
+  <transmission name="l_b_motor_transmission">
+    <type>transmission_interface/SimpleTransmission</type>
+    <joint name="l_b_motor_joint">
+      <hardwareInterface>EffortJointInterface</hardwareInterface>
+    </joint>
+    <actuator name="l_b_m1">
+      <hardwareInterface>EffortJointInterface</hardwareInterface>
+      <mechanicalReduction>1</mechanicalReduction>
+    </actuator>
+  </transmission>
+  <transmission name="r_f_motor_transmission">
+    <type>transmission_interface/SimpleTransmission</type>
+    <joint name="r_f_motor_joint">
+      <hardwareInterface>EffortJointInterface</hardwareInterface>
+    </joint>
+    <actuator name="r_f_m1">
+      <hardwareInterface>EffortJointInterface</hardwareInterface>
+      <mechanicalReduction>1</mechanicalReduction>
+    </actuator>
+  </transmission>
+  <transmission name="r_b_motor">
+    <type>transmission_interface/SimpleTransmission</type>
+    <joint name="r_b_motor_joint">
+      <hardwareInterface>EffortJointInterface</hardwareInterface>
+    </joint>
+    <actuator name="r_b_m1">
+      <hardwareInterface>EffortJointInterface</hardwareInterface>
+      <mechanicalReduction>1</mechanicalReduction>
+    </actuator>
+  </transmission>
+  <transmission name="l_f_h_motor_transmission">
+    <type>transmission_interface/SimpleTransmission</type>
+    <joint name="l_f_h_motor_joint">
+      <hardwareInterface>EffortJointInterface</hardwareInterface>
+    </joint>
+    <actuator name="l_f_h_m2">
+      <hardwareInterface>EffortJointInterface</hardwareInterface>
+      <mechanicalReduction>1</mechanicalReduction>
+    </actuator>
+  </transmission>
+  <transmission name="l_b_h_motor_transmission">
+    <type>transmission_interface/SimpleTransmission</type>
+    <joint name="l_b_h_motor_joint">
+      <hardwareInterface>EffortJointInterface</hardwareInterface>
+    </joint>
+    <actuator name="l_b_h_m2">
+      <hardwareInterface>EffortJointInterface</hardwareInterface>
+      <mechanicalReduction>1</mechanicalReduction>
+    </actuator>
+  </transmission>
+  <transmission name="r_f_h_motor_transmission">
+    <type>transmission_interface/SimpleTransmission</type>
+    <joint name="r_f_h_motor_joint">
+      <hardwareInterface>EffortJointInterface</hardwareInterface>
+    </joint>
+    <actuator name="r_f_h_m2">
+      <hardwareInterface>EffortJointInterface</hardwareInterface>
+      <mechanicalReduction>1</mechanicalReduction>
+    </actuator>
+  </transmission>
+  <transmission name="r_b_h_motor_transmission">
+    <type>transmission_interface/SimpleTransmission</type>
+    <joint name="r_b_h_motor_joint">
+      <hardwareInterface>EffortJointInterface</hardwareInterface>
+    </joint>
+    <actuator name="r_b_h_m2">
+      <hardwareInterface>EffortJointInterface</hardwareInterface>
+      <mechanicalReduction>1</mechanicalReduction>
+    </actuator>
+  </transmission-->
+<!--#######################################################################################################################################-->
 <!--contact_sensor_torso_base-->
 <gazebo reference="torso_base">
@@ -597,3 +627,39 @@
   </plugin>
 </gazebo>
+<!--################################################hokuyo_sensor_plugin##################################-->
+<gazebo reference="hokuyo_link">
+    <sensor type="ray" name="head_hokuyo_sensor">
+        <pose>0 0 0 0 0 0</pose>
+        <visualize>true</visualize>
+        <update_rate>60</update_rate>
+        <ray>
+            <scan>
+            <horizontal>
+                <samples>720</samples>
+                <resolution>1</resolution>
+                <min_angle>-0.785</min_angle>
+                <max_angle>0.785</max_angle>
+            </horizontal>
+            </scan>
+            <range>
+                <min>0.10</min>
+                <max>5.0</max>
+                <resolution>0.01</resolution>
+            </range>
+            <noise>
+                <type>gaussian</type>
+                <!-- Noise parameters based on published spec for Hokuyo laser
+                    achieving "+-30mm" accuracy at range < 10m.  A mean of 0.0m and
+                    stddev of 0.01m will put 99.7% of samples within 0.03m of the true
+                    reading. -->
+                <mean>0.0</mean>
+                <stddev>0.01</stddev>
+            </noise>
+        </ray>
+        <plugin name="laser" filename="libgazebo_ros_laser.so">
+            <topicName>/scan</topicName>
+            <frameName>hokuyo_link</frameName>
+        </plugin>
+    </sensor>
+</gazebo>
 </robot>
