Commit message: urdf modified

File: insect_description/urdf/insect.urdf.xacro (robot description, xacro)
@@ -17,5 +17,5 @@
   <origin xyz="0 0 0" rpy="0 0 0"/>
   <geometry>
-    <mesh filename="file:///home/rit/catkin_ws2/src/insect_robot/insect_description/meshes/torso_v1.dae"/>
+    <mesh filename="package://insect_description/meshes/torso_v1.dae"/>
   </geometry>
 </collision>
@@ -23,5 +23,5 @@
   <origin xyz="0 0 0" rpy="0 0 0"/>
   <geometry>
-    <mesh filename="file:///home/rit/catkin_ws2/src/insect_robot/insect_description/meshes/torso_v1.dae"/>
+    <mesh filename="package://insect_description/meshes/torso_v1.dae"/>
   </geometry>
 </visual>
@@ -47,5 +47,5 @@
       <origin xyz="0 0 0" rpy="0 -0.5 -1.5"/>
         <geometry>
-          <mesh filename="file:///home/rit/catkin_ws2/src/insect_robot/insect_description/meshes/motor_v1.dae"/>
+          <mesh filename="package://insect_description/meshes/motor_v1.dae"/>
         </geometry>
       </collision>
@@ -53,5 +53,5 @@
         <origin xyz="0 0 0" rpy="0 -0.5 -1.4"/>
         <geometry>
-          <mesh filename="file:///home/rit/catkin_ws2/src/insect_robot/insect_description/meshes/motor_v1.dae"/>
+          <mesh filename="package://insect_description/meshes/motor_v1.dae"/>
         </geometry>
       </visual>
@@ -62,5 +62,5 @@
         <origin xyz="0 0 0" rpy="0 -0.5 1.5"/>
           <geometry>
-            <mesh filename="file:///home/rit/catkin_ws2/src/insect_robot/insect_description/meshes/motor_v1.dae"/>
+            <mesh filename="package://insect_description/meshes/motor_v1.dae"/>
           </geometry>
         </collision>
@@ -68,5 +68,5 @@
           <origin xyz="0 0 0" rpy="0 -0.5 1.5"/>
           <geometry>
-            <mesh filename="file:///home/rit/catkin_ws2/src/insect_robot/insect_description/meshes/motor_v1.dae"/>
+            <mesh filename="package://insect_description/meshes/motor_v1.dae"/>
           </geometry>
         </visual>
@@ -77,5 +77,5 @@
           <origin xyz="0 0 0" rpy="0 -0.5 -1.5"/>
             <geometry>
-              <mesh filename="file:///home/rit/catkin_ws2/src/insect_robot/insect_description/meshes/motor_v1.dae"/>
+              <mesh filename="package://insect_description/meshes/motor_v1.dae"/>
             </geometry>
           </collision>
@@ -83,5 +83,5 @@
             <origin xyz="0 0 0" rpy="0 -0.5 -1.5"/>
             <geometry>
-              <mesh filename="file:///home/rit/catkin_ws2/src/insect_robot/insect_description/meshes/motor_v1.dae"/>
+              <mesh filename="package://insect_description/meshes/motor_v1.dae"/>
             </geometry>
           </visual>
@@ -92,5 +92,5 @@
             <origin xyz="0 0 0" rpy="0 -0.5 1.5"/>
               <geometry>
-                <mesh filename="file:///home/rit/catkin_ws2/src/insect_robot/insect_description/meshes/motor_v1.dae"/>
+                <mesh filename="package://insect_description/meshes/motor_v1.dae"/>
               </geometry>
             </collision>
@@ -98,5 +98,5 @@
               <origin xyz="0 0 0" rpy="0 -0.5 1.5"/>
               <geometry>
-                <mesh filename="file:///home/rit/catkin_ws2/src/insect_robot/insect_description/meshes/motor_v1.dae"/>
+                <mesh filename="package://insect_description/meshes/motor_v1.dae"/>
               </geometry>
             </visual>
@@ -107,5 +107,5 @@
               <origin xyz="0 0 0" rpy="0 -0.5 -1.5"/>
                 <geometry>
-                  <mesh filename="file:///home/rit/catkin_ws2/src/insect_robot/insect_description/meshes/hip_v1.dae"/>
+                  <mesh filename="package://insect_description/meshes/hip_v1.dae"/>
                 </geometry>
               </collision>
@@ -113,5 +113,5 @@
                 <origin xyz="0 0 0" rpy="0 -0.5 -1.5"/>
                 <geometry>
-                  <mesh filename="file:///home/rit/catkin_ws2/src/insect_robot/insect_description/meshes/hip_v1.dae"/>
+                  <mesh filename="package://insect_description/meshes/hip_v1.dae"/>
                 </geometry>
               </visual>
@@ -122,5 +122,5 @@
                 <origin xyz="0 0 0" rpy="0 -0.5 1.5"/>
                   <geometry>
-                    <mesh filename="file:///home/rit/catkin_ws2/src/insect_robot/insect_description/meshes/hip_v1.dae"/>
+                    <mesh filename="package://insect_description/meshes/hip_v1.dae"/>
                   </geometry>
                 </collision>
@@ -128,5 +128,5 @@
                   <origin xyz="0 0 0" rpy="0 -0.5 1.5"/>
                   <geometry>
-                    <mesh filename="file:///home/rit/catkin_ws2/src/insect_robot/insect_description/meshes/hip_v1.dae"/>
+                    <mesh filename="package://insect_description/meshes/hip_v1.dae"/>
                   </geometry>
                 </visual>
@@ -137,5 +137,5 @@
                   <origin xyz="0 0 0" rpy="0 -0.5 -1.5"/>
                     <geometry>
-                      <mesh filename="file:///home/rit/catkin_ws2/src/insect_robot/insect_description/meshes/hip_v1.dae"/>
+                      <mesh filename="package://insect_description/meshes/hip_v1.dae"/>
                     </geometry>
                   </collision>
@@ -143,5 +143,5 @@
                     <origin xyz="0 0 0" rpy="0 -0.5 -1.5"/>
                     <geometry>
-                      <mesh filename="file:///home/rit/catkin_ws2/src/insect_robot/insect_description/meshes/hip_v1.dae"/>
+                      <mesh filename="package://insect_description/meshes/hip_v1.dae"/>
                     </geometry>
                   </visual>
@@ -152,5 +152,5 @@
                     <origin xyz="0 0 0" rpy="0 -0.5 1.5"/>
                       <geometry>
-                        <mesh filename="file:///home/rit/catkin_ws2/src/insect_robot/insect_description/meshes/hip_v1.dae"/>
+                        <mesh filename="package://insect_description/meshes/hip_v1.dae"/>
                       </geometry>
                     </collision>
@@ -158,5 +158,5 @@
                       <origin xyz="0 0 0" rpy="0 -0.5 1.5"/>
                       <geometry>
-                        <mesh filename="file:///home/rit/catkin_ws2/src/insect_robot/insect_description/meshes/hip_v1.dae"/>
+                        <mesh filename="package://insect_description/meshes/hip_v1.dae"/>
                       </geometry>
                     </visual>
@@ -167,5 +167,5 @@
                       <origin xyz="0 0 0" rpy="0 -3.4 -1.5"/>
                         <geometry>
-                          <mesh filename="file:///home/rit/catkin_ws2/src/insect_robot/insect_description/meshes/motor_h_v1.dae"/>
+                          <mesh filename="package://insect_description/meshes/motor_h_v1.dae"/>
                         </geometry>
                       </collision>
@@ -173,5 +173,5 @@
                         <origin xyz="0 0 0" rpy="0 -3.4 -1.5"/>
                         <geometry>
-                          <mesh filename="file:///home/rit/catkin_ws2/src/insect_robot/insect_description/meshes/motor_h_v1.dae"/>
+                          <mesh filename="package://insect_description/meshes/motor_h_v1.dae"/>
                         </geometry>
                       </visual>
@@ -182,5 +182,5 @@
                         <origin xyz="0 0 0" rpy="0 -3.4 -1.5"/>
                           <geometry>
-                            <mesh filename="file:///home/rit/catkin_ws2/src/insect_robot/insect_description/meshes/motor_h_v1.dae"/>
+                            <mesh filename="package://insect_description/meshes/motor_h_v1.dae"/>
                           </geometry>
                         </collision>
@@ -188,5 +188,5 @@
                           <origin xyz="0 0 0" rpy="0 -3.4 1.5"/>
                           <geometry>
-                            <mesh filename="file:///home/rit/catkin_ws2/src/insect_robot/insect_description/meshes/motor_h_v1.dae"/>
+                            <mesh filename="package://insect_description/meshes/motor_h_v1.dae"/>
                           </geometry>
                         </visual>
@@ -197,5 +197,5 @@
                           <origin xyz="0 0 0" rpy="0 -3.4 -1.5"/>
                             <geometry>
-                              <mesh filename="file:///home/rit/catkin_ws2/src/insect_robot/insect_description/meshes/motor_h_v1.dae"/>
+                              <mesh filename="package://insect_description/meshes/motor_h_v1.dae"/>
                             </geometry>
                           </collision>
@@ -203,5 +203,5 @@
                             <origin xyz="0 0 0" rpy="0 -3.4 -1.5"/>
                             <geometry>
-                              <mesh filename="file:///home/rit/catkin_ws2/src/insect_robot/insect_description/meshes/motor_h_v1.dae"/>
+                              <mesh filename="package://insect_description/meshes/motor_h_v1.dae"/>
                             </geometry>
                           </visual>
@@ -212,5 +212,5 @@
                             <origin xyz="0 0 0" rpy="0 -3.4 -1.5"/>
                               <geometry>
-                                <mesh filename="file:///home/rit/catkin_ws2/src/insect_robot/insect_description/meshes/motor_h_v1.dae"/>
+                                <mesh filename="package://insect_description/meshes/motor_h_v1.dae"/>
                               </geometry>
                             </collision>
@@ -218,5 +218,5 @@
                               <origin xyz="0 0 0" rpy="0 -3.4 1.5"/>
                               <geometry>
-                                <mesh filename="file:///home/rit/catkin_ws2/src/insect_robot/insect_description/meshes/motor_h_v1.dae"/>
+                                <mesh filename="package://insect_description/meshes/motor_h_v1.dae"/>
                               </geometry>
                             </visual>
@@ -227,5 +227,5 @@
                               <origin xyz="0 0 0" rpy="0 0 -1.5"/>
                                 <geometry>
-                                  <mesh filename="file:///home/rit/catkin_ws2/src/insect_robot/insect_description/meshes/leg_v1.dae"/>
+                                  <mesh filename="package://insect_description/meshes/leg_v1.dae"/>
                                 </geometry>
                               </collision>
@@ -233,5 +233,5 @@
                                 <origin xyz="0 0 0" rpy="0 0 -1.5"/>
                                 <geometry>
-                                  <mesh filename="file:///home/rit/catkin_ws2/src/insect_robot/insect_description/meshes/leg_v1.dae"/>
+                                  <mesh filename="package://insect_description/meshes/leg_v1.dae"/>
                                 </geometry>
                               </visual>
@@ -242,5 +242,5 @@
                                 <origin xyz="0 0 0" rpy="0 0 -1.5"/>
                                   <geometry>
-                                    <mesh filename="file:///home/rit/catkin_ws2/src/insect_robot/insect_description/meshes/leg_v1.dae"/>
+                                    <mesh filename="package://insect_description/meshes/leg_v1.dae"/>
                                   </geometry>
                                 </collision>
@@ -248,5 +248,5 @@
                                   <origin xyz="0 0 0" rpy="0 0 -1.5"/>
                                   <geometry>
-                                    <mesh filename="file:///home/rit/catkin_ws2/src/insect_robot/insect_description/meshes/leg_v1.dae"/>
+                                    <mesh filename="package://insect_description/meshes/leg_v1.dae"/>
                                   </geometry>
                                 </visual>
@@ -257,5 +257,5 @@
                                   <origin xyz="0 0 0" rpy="0 0 1.5"/>
                                     <geometry>
-                                      <mesh filename="file:///home/rit/catkin_ws2/src/insect_robot/insect_description/meshes/leg_v1.dae"/>
+                                      <mesh filename="package://insect_description/meshes/leg_v1.dae"/>
                                     </geometry>
                                   </collision>
@@ -263,5 +263,5 @@
                                     <origin xyz="0 0 0" rpy="0 0 1.5"/>
                                     <geometry>
-                                      <mesh filename="file:///home/rit/catkin_ws2/src/insect_robot/insect_description/meshes/leg_v1.dae"/>
+                                      <mesh filename="package://insect_description/meshes/leg_v1.dae"/>
                                     </geometry>
                                   </visual>
@@ -272,5 +272,5 @@
                                     <origin xyz="0 0 0" rpy="0 0 1.5"/>
                                       <geometry>
-                                        <mesh filename="file:///home/rit/catkin_ws2/src/insect_robot/insect_description/meshes/leg_v1.dae"/>
+                                        <mesh filename="package://insect_description/meshes/leg_v1.dae"/>
                                       </geometry>
                                     </collision>
@@ -278,5 +278,5 @@
                                       <origin xyz="0 0 0" rpy="0 0 1.5"/>
                                       <geometry>
-                                        <mesh filename="file:///home/rit/catkin_ws2/src/insect_robot/insect_description/meshes/leg_v1.dae"/>
+                                        <mesh filename="package://insect_description/meshes/leg_v1.dae"/>
                                       </geometry>
                                     </visual>
@@ -284,5 +284,5 @@
                                   </link>
 <!--############################################################################################################################-->
-                                  <link name="hokuyo_link">
+                                  <!--link name="hokuyo_link">
                                       <collision>
                                           <origin xyz="0 0 0" rpy="0 0 0"/>
@@ -291,13 +291,13 @@
                                           </geometry>
                                       </collision>     <origin xyz="0 0 0" rpy="0 0 0"/>
-                                          <geometry>
-                                              <!--mesh filename="package://insect/meshes/hokuyo.dae"/-->
-                                              <mesh filename="file:///home/rit/catkin_ws2/src/insect_robot/insect_description/meshes/hokuyo.dae"/>
+                                          <geometry-->
+                                              <!--mesh filename="package://://insect/meshes/hokuyo.dae"/-->
+                                              <!--mesh filename="package://insect_description/meshes/hokuyo.dae"/>
                                           </geometry>
                                       <visual>
                                           <origin xyz="0 0 0" rpy="0 0 0"/>
-                                          <geometry>
-                                              <!--mesh filename="package://insect/meshes/hokuyo.dae"/-->
-                                              <mesh filename="file:///home/rit/catkin_ws2/src/insect_robot/insect_description/meshes/hokuyo.dae"/>
+                                          <geometry-->
+                                              <!--mesh filename="package://://insect/meshes/hokuyo.dae"/-->
+                                              <!--mesh filename="package://insect_description/meshes/hokuyo.dae"/>
                                           </geometry>
                                       </visual>
@@ -307,5 +307,5 @@
                                           <inertia ixx="1e-6" ixy="0" ixz="0" iyy="1e-6" iyz="0" izz="1e-6" />
                                       </inertial>
-                                  </link>
+                                  </link-->
 <!--#########################################################################################################################################-->
 <!-- Joint properties -->
@@ -315,9 +315,9 @@
 <xacro:property name="joint_velocity" value="0.524"/>
 <!--######################################################################################################################################-->
-<joint name="hokuyo_joint" type="fixed">
-    <origin xyz="0.04 0 0.08" rpy="0 0 0"/>
+<!--joint name="hokuyo_joint" type="fixed">
+    <origin xyz="0 0 0.08" rpy="0 0 0"/>
     <parent link="torso_base"/>
     <child link="hokuyo_link"/>
-</joint>
+</joint-->
 <joint name="world_joint"  type="fixed">
   <origin xyz="0 0 0.30" rpy="0 0 0" />
@@ -325,6 +325,4 @@
   <child link="torso_base"/>
   <axis xyz="0 1 0" rpy="0 0 0"/>
-  <limit effort="10000" velocity="1000"/>
-  <joint_properties damping="1.0" friction="1.0"/>
 </joint>
 <!--IMU sensor joint-->
@@ -340,6 +338,4 @@
   <child link="l_f_motor"/>
   <axis xyz="0 1 0" rpy="0 0 0"/>
-  <limit effort="10000" velocity="1000"/>
-  <joint_properties damping="1.0" friction="1.0"/>
 </joint>
 <joint name="r_f_motor_joint"  type="fixed">
@@ -348,6 +344,4 @@
   <child link="r_f_motor"/>
   <axis xyz="0 1 0" rpy="0 0 0"/>
-  <limit effort="10000" velocity="1000"/>
-  <joint_properties damping="1.0" friction="1.0"/>
 </joint>
 <joint name="l_b_motor_joint"  type="fixed">
@@ -356,6 +350,4 @@
   <child link="l_b_motor"/>
   <axis xyz="0 1 0" rpy="0 0 0"/>
-  <limit effort="10000" velocity="1000"/>
-  <joint_properties damping="1.0" friction="1.0"/>
 </joint>
 <joint name="r_b_motor_joint"  type="fixed">
@@ -364,6 +356,4 @@
   <child link="r_b_motor"/>
   <axis xyz="0 1 0" rpy="0 0 0"/>
-  <limit effort="10000" velocity="1000"/>
-  <joint_properties damping="1.0" friction="1.0"/>
 </joint>
 <joint name="l_f_hip_joint"  type="fixed">
@@ -372,6 +362,4 @@
   <child link="l_f_hip"/>
   <axis xyz="0 1 0" rpy="0 0 0"/>
-  <limit effort="10000" velocity="1000"/>
-  <joint_properties damping="1.0" friction="1.0"/>
 </joint>
 <joint name="r_f_hip_joint"  type="fixed">
@@ -380,6 +368,4 @@
   <child link="r_f_hip"/>
   <axis xyz="0 1 0" rpy="0 0 0"/>
-  <limit effort="10000" velocity="1000"/>
-  <joint_properties damping="1.0" friction="1.0"/>
 </joint>
 <joint name="l_b_hip_joint"  type="fixed">
@@ -388,6 +374,4 @@
   <child link="l_b_hip"/>
   <axis xyz="0 1 0" rpy="0 0 0"/>
-  <limit effort="10000" velocity="1000"/>
-  <joint_properties damping="1.0" friction="1.0"/>
 </joint>
 <joint name="r_b_hip_joint"  type="fixed">
@@ -396,6 +380,4 @@
   <child link="r_b_hip"/>
   <axis xyz="0 1 0" rpy="0 0 0"/>
-  <limit effort="10000" velocity="1000"/>
-  <joint_properties damping="1.0" friction="1.0"/>
 </joint>
 <joint name="l_f_h_motor_joint"  type="fixed">
@@ -404,6 +386,4 @@
   <child link="l_f_h_motor"/>
   <axis xyz="0 1 0" rpy="0 0 0"/>
-  <limit effort="10000" velocity="1000"/>
-  <joint_properties damping="1.0" friction="1.0"/>
 </joint>
 <joint name="r_f_h_motor_joint"  type="fixed">
@@ -412,6 +392,4 @@
   <child link="r_f_h_motor"/>
   <axis xyz="0 1 0" rpy="0 0 0"/>
-  <limit effort="10000" velocity="1000"/>
-  <joint_properties damping="1.0" friction="1.0"/>
 </joint>
 <joint name="l_b_h_motor_joint"  type="fixed">
@@ -420,6 +398,4 @@
   <child link="l_b_h_motor"/>
   <axis xyz="0 1 0" rpy="0 0 0"/>
-  <limit effort="10000" velocity="1000"/>
-  <joint_properties damping="1.0" friction="1.0"/>
 </joint>
 <joint name="r_b_h_motor_joint"  type="fixed">
@@ -428,6 +404,4 @@
   <child link="r_b_h_motor"/>
   <axis xyz="0 1 0" rpy="0 0 0"/>
-  <limit effort="10000" velocity="1000"/>
-  <joint_properties damping="1.0" friction="1.0"/>
 </joint>
 <joint name="l_f_leg_joint"  type="fixed">
@@ -436,6 +410,4 @@
   <child link="l_f_leg"/>
   <axis xyz="0 1 0" rpy="0 0 0"/>
-  <limit effort="10000" velocity="1000"/>
-  <joint_properties damping="1.0" friction="1.0"/>
 </joint>
 <joint name="l_b_leg_joint"  type="fixed">
@@ -444,6 +416,4 @@
   <child link="l_b_leg"/>
   <axis xyz="0 1 0" rpy="0 0 0"/>
-  <limit effort="10000" velocity="1000"/>
-  <joint_properties damping="1.0" friction="1.0"/>
 </joint>
 <joint name="r_f_leg_joint"  type="fixed">
@@ -452,6 +422,4 @@
   <child link="r_f_leg"/>
   <axis xyz="0 1 0" rpy="0 0 0"/>
-  <limit effort="10000" velocity="1000"/>
-  <joint_properties damping="1.0" friction="1.0"/>
 </joint>
 <joint name="r_b_leg_joint"  type="fixed">
@@ -460,9 +428,7 @@
   <child link="r_b_leg"/>
   <axis xyz="0 1 0" rpy="0 0 0"/>
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