Commit message: modification in urdf

File: insect_description/urdf/insect.urdf.xacro (robot description, xacro)
@@ -1,3 +1,3 @@
-<?xml version='1.0'?>
+<?xml version="1.0" encoding="UTF-8"?>
 <robot name="insect" xmlns:xacro="http://www.ros.org/wiki/xacro">
 <!--##################################################################################################################################-->
@@ -7,4 +7,5 @@
 <xacro:macro name="default_inertial" params="mass">
    <inertial>
+     <origin xyz="0.0 0.0 0.0" rpy="0.0 0.0 0.0" />
      <mass value="${mass}" />
      <inertia ixx="1.0" ixy="0.0" ixz="0.0" iyy="1.0" iyz="0.0" izz="1.0" />
@@ -17,5 +18,9 @@
   <origin xyz="0 0 0" rpy="0 0 0"/>
   <geometry>
+<<<<<<< HEAD
+    <mesh filename="package://insect_description/meshes/torso_v1.dae" />
+=======
     <mesh filename="package://insect_description/meshes/torso_v1.dae"/>
+>>>>>>> 91e1ca3aa603a8a23207d7aa177f3fa7cca5ff34
   </geometry>
 </collision>
@@ -23,5 +28,9 @@
   <origin xyz="0 0 0" rpy="0 0 0"/>
   <geometry>
+<<<<<<< HEAD
+    <mesh filename="package://insect_description/meshes/torso_v1.dae" />
+=======
     <mesh filename="package://insect_description/meshes/torso_v1.dae"/>
+>>>>>>> 91e1ca3aa603a8a23207d7aa177f3fa7cca5ff34
   </geometry>
 </visual>
@@ -47,5 +56,9 @@
       <origin xyz="0 0 0" rpy="0 -0.5 -1.5"/>
         <geometry>
+<<<<<<< HEAD
+          <mesh filename="package://insect_description/meshes/motor_v1.dae" />
+=======
           <mesh filename="package://insect_description/meshes/motor_v1.dae"/>
+>>>>>>> 91e1ca3aa603a8a23207d7aa177f3fa7cca5ff34
         </geometry>
       </collision>
@@ -53,14 +66,22 @@
         <origin xyz="0 0 0" rpy="0 -0.5 -1.4"/>
         <geometry>
+<<<<<<< HEAD
+          <mesh filename="package://insect_description/meshes/motor_v1.dae" />
+=======
           <mesh filename="package://insect_description/meshes/motor_v1.dae"/>
+>>>>>>> 91e1ca3aa603a8a23207d7aa177f3fa7cca5ff34
         </geometry>
       </visual>
       <xacro:default_inertial mass="0.2"/>
     </link>
-    <link name= "r_f_motor">
+    <!--link name= "r_f_motor">
       <collision name="collision">
         <origin xyz="0 0 0" rpy="0 -0.5 1.5"/>
           <geometry>
+<<<<<<< HEAD
+            <mesh filename="package://insect_description/meshes/motor_v1.dae" />
+=======
             <mesh filename="package://insect_description/meshes/motor_v1.dae"/>
+>>>>>>> 91e1ca3aa603a8a23207d7aa177f3fa7cca5ff34
           </geometry>
         </collision>
@@ -68,5 +89,9 @@
           <origin xyz="0 0 0" rpy="0 -0.5 1.5"/>
           <geometry>
+<<<<<<< HEAD
+            <mesh filename="package://insect_description/meshes/motor_v1.dae" />
+=======
             <mesh filename="package://insect_description/meshes/motor_v1.dae"/>
+>>>>>>> 91e1ca3aa603a8a23207d7aa177f3fa7cca5ff34
           </geometry>
         </visual>
@@ -77,5 +102,9 @@
           <origin xyz="0 0 0" rpy="0 -0.5 -1.5"/>
             <geometry>
+<<<<<<< HEAD
+              <mesh filename="package://insect_description/meshes/motor_v1.dae" />
+=======
               <mesh filename="package://insect_description/meshes/motor_v1.dae"/>
+>>>>>>> 91e1ca3aa603a8a23207d7aa177f3fa7cca5ff34
             </geometry>
           </collision>
@@ -83,5 +112,9 @@
             <origin xyz="0 0 0" rpy="0 -0.5 -1.5"/>
             <geometry>
+<<<<<<< HEAD
+              <mesh filename="package://insect_description/meshes/motor_v1.dae" />
+=======
               <mesh filename="package://insect_description/meshes/motor_v1.dae"/>
+>>>>>>> 91e1ca3aa603a8a23207d7aa177f3fa7cca5ff34
             </geometry>
           </visual>
@@ -92,5 +125,9 @@
             <origin xyz="0 0 0" rpy="0 -0.5 1.5"/>
               <geometry>
+<<<<<<< HEAD
+                <mesh filename="package://insect_description/meshes/motor_v1.dae" />
+=======
                 <mesh filename="package://insect_description/meshes/motor_v1.dae"/>
+>>>>>>> 91e1ca3aa603a8a23207d7aa177f3fa7cca5ff34
               </geometry>
             </collision>
@@ -98,14 +135,22 @@
               <origin xyz="0 0 0" rpy="0 -0.5 1.5"/>
               <geometry>
+<<<<<<< HEAD
+                <mesh filename="package://insect_description/meshes/motor_v1.dae" />
+=======
                 <mesh filename="package://insect_description/meshes/motor_v1.dae"/>
+>>>>>>> 91e1ca3aa603a8a23207d7aa177f3fa7cca5ff34
               </geometry>
             </visual>
             <xacro:default_inertial mass="0.2"/>
-          </link>
+          </link-->
           <link name= "l_f_hip">
             <collision name="collision">
               <origin xyz="0 0 0" rpy="0 -0.5 -1.5"/>
                 <geometry>
+<<<<<<< HEAD
+                  <mesh filename="package://insect_description/meshes/hip_v1.dae" />
+=======
                   <mesh filename="package://insect_description/meshes/hip_v1.dae"/>
+>>>>>>> 91e1ca3aa603a8a23207d7aa177f3fa7cca5ff34
                 </geometry>
               </collision>
@@ -113,14 +158,22 @@
                 <origin xyz="0 0 0" rpy="0 -0.5 -1.5"/>
                 <geometry>
+<<<<<<< HEAD
+                  <mesh filename="package://insect_description/meshes/hip_v1.dae" />
+=======
                   <mesh filename="package://insect_description/meshes/hip_v1.dae"/>
+>>>>>>> 91e1ca3aa603a8a23207d7aa177f3fa7cca5ff34
                 </geometry>
               </visual>
               <xacro:default_inertial mass="0.4"/>
             </link>
-            <link name= "r_f_hip">
+            <!--link name= "r_f_hip">
               <collision name="collision">
                 <origin xyz="0 0 0" rpy="0 -0.5 1.5"/>
                   <geometry>
+<<<<<<< HEAD
+                    <mesh filename="package://insect_description/meshes/hip_v1.dae" />
+=======
                     <mesh filename="package://insect_description/meshes/hip_v1.dae"/>
+>>>>>>> 91e1ca3aa603a8a23207d7aa177f3fa7cca5ff34
                   </geometry>
                 </collision>
@@ -128,5 +181,9 @@
                   <origin xyz="0 0 0" rpy="0 -0.5 1.5"/>
                   <geometry>
+<<<<<<< HEAD
+                    <mesh filename="package://insect_description/meshes/hip_v1.dae" />
+=======
                     <mesh filename="package://insect_description/meshes/hip_v1.dae"/>
+>>>>>>> 91e1ca3aa603a8a23207d7aa177f3fa7cca5ff34
                   </geometry>
                 </visual>
@@ -137,5 +194,9 @@
                   <origin xyz="0 0 0" rpy="0 -0.5 -1.5"/>
                     <geometry>
+<<<<<<< HEAD
+                      <mesh filename="package://insect_description/meshes/hip_v1.dae" />
+=======
                       <mesh filename="package://insect_description/meshes/hip_v1.dae"/>
+>>>>>>> 91e1ca3aa603a8a23207d7aa177f3fa7cca5ff34
                     </geometry>
                   </collision>
@@ -143,5 +204,9 @@
                     <origin xyz="0 0 0" rpy="0 -0.5 -1.5"/>
                     <geometry>
+<<<<<<< HEAD
+                      <mesh filename="package://insect_description/meshes/hip_v1.dae" />
+=======
                       <mesh filename="package://insect_description/meshes/hip_v1.dae"/>
+>>>>>>> 91e1ca3aa603a8a23207d7aa177f3fa7cca5ff34
                     </geometry>
                   </visual>
@@ -152,5 +217,9 @@
                     <origin xyz="0 0 0" rpy="0 -0.5 1.5"/>
                       <geometry>
+<<<<<<< HEAD
+                        <mesh filename="package://insect_description/meshes/hip_v1.dae" />
+=======
                         <mesh filename="package://insect_description/meshes/hip_v1.dae"/>
+>>>>>>> 91e1ca3aa603a8a23207d7aa177f3fa7cca5ff34
                       </geometry>
                     </collision>
@@ -158,5 +227,9 @@
                       <origin xyz="0 0 0" rpy="0 -0.5 1.5"/>
                       <geometry>
+<<<<<<< HEAD
+                        <mesh filename="package://insect_description/meshes/hip_v1.dae" />
+=======
                         <mesh filename="package://insect_description/meshes/hip_v1.dae"/>
+>>>>>>> 91e1ca3aa603a8a23207d7aa177f3fa7cca5ff34
                       </geometry>
                     </visual>
@@ -167,5 +240,9 @@
                       <origin xyz="0 0 0" rpy="0 -3.4 -1.5"/>
                         <geometry>
+<<<<<<< HEAD
+                          <mesh filename="package://insect_description/meshes/motor_h_v1.dae" />
+=======
                           <mesh filename="package://insect_description/meshes/motor_h_v1.dae"/>
+>>>>>>> 91e1ca3aa603a8a23207d7aa177f3fa7cca5ff34
                         </geometry>
                       </collision>
@@ -173,5 +250,9 @@
                         <origin xyz="0 0 0" rpy="0 -3.4 -1.5"/>
                         <geometry>
+<<<<<<< HEAD
+                          <mesh filename="package://insect_description/meshes/motor_h_v1.dae" />
+=======
                           <mesh filename="package://insect_description/meshes/motor_h_v1.dae"/>
+>>>>>>> 91e1ca3aa603a8a23207d7aa177f3fa7cca5ff34
                         </geometry>
                       </visual>
@@ -182,5 +263,9 @@
                         <origin xyz="0 0 0" rpy="0 -3.4 -1.5"/>
                           <geometry>
+<<<<<<< HEAD
+                            <mesh filename="package://insect_description/meshes/motor_h_v1.dae" />
+=======
                             <mesh filename="package://insect_description/meshes/motor_h_v1.dae"/>
+>>>>>>> 91e1ca3aa603a8a23207d7aa177f3fa7cca5ff34
                           </geometry>
                         </collision>
@@ -188,5 +273,9 @@
                           <origin xyz="0 0 0" rpy="0 -3.4 1.5"/>
                           <geometry>
+<<<<<<< HEAD
+                            <mesh filename="package://insect_description/meshes/motor_h_v1.dae" />
+=======
                             <mesh filename="package://insect_description/meshes/motor_h_v1.dae"/>
+>>>>>>> 91e1ca3aa603a8a23207d7aa177f3fa7cca5ff34
                           </geometry>
                         </visual>
@@ -197,5 +286,9 @@
                           <origin xyz="0 0 0" rpy="0 -3.4 -1.5"/>
                             <geometry>
+<<<<<<< HEAD
+                              <mesh filename="package://insect_description/meshes/motor_h_v1.dae" />
+=======
                               <mesh filename="package://insect_description/meshes/motor_h_v1.dae"/>
+>>>>>>> 91e1ca3aa603a8a23207d7aa177f3fa7cca5ff34
                             </geometry>
                           </collision>
@@ -203,5 +296,9 @@
                             <origin xyz="0 0 0" rpy="0 -3.4 -1.5"/>
                             <geometry>
+<<<<<<< HEAD
+                              <mesh filename="package://insect_description/meshes/motor_h_v1.dae" />
+=======
                               <mesh filename="package://insect_description/meshes/motor_h_v1.dae"/>
+>>>>>>> 91e1ca3aa603a8a23207d7aa177f3fa7cca5ff34
                             </geometry>
                           </visual>
@@ -212,5 +309,9 @@
                             <origin xyz="0 0 0" rpy="0 -3.4 -1.5"/>
                               <geometry>
+<<<<<<< HEAD
+                                <mesh filename="package://insect_description/meshes/motor_h_v1.dae" />
+=======
                                 <mesh filename="package://insect_description/meshes/motor_h_v1.dae"/>
+>>>>>>> 91e1ca3aa603a8a23207d7aa177f3fa7cca5ff34
                               </geometry>
                             </collision>
@@ -218,5 +319,9 @@
                               <origin xyz="0 0 0" rpy="0 -3.4 1.5"/>
                               <geometry>
+<<<<<<< HEAD
+                                <mesh filename="package://insect_description/meshes/motor_h_v1.dae" />
+=======
                                 <mesh filename="package://insect_description/meshes/motor_h_v1.dae"/>
+>>>>>>> 91e1ca3aa603a8a23207d7aa177f3fa7cca5ff34
                               </geometry>
                             </visual>
@@ -227,5 +332,9 @@
                               <origin xyz="0 0 0" rpy="0 0 -1.5"/>
                                 <geometry>
+<<<<<<< HEAD
+                                  <mesh filename="package://insect_description/meshes/leg_v1.dae" />
+=======
                                   <mesh filename="package://insect_description/meshes/leg_v1.dae"/>
+>>>>>>> 91e1ca3aa603a8a23207d7aa177f3fa7cca5ff34
                                 </geometry>
                               </collision>
@@ -233,5 +342,9 @@
                                 <origin xyz="0 0 0" rpy="0 0 -1.5"/>
                                 <geometry>
+<<<<<<< HEAD
+                                  <mesh filename="package://insect_description/meshes/leg_v1.dae" />
+=======
                                   <mesh filename="package://insect_description/meshes/leg_v1.dae"/>
+>>>>>>> 91e1ca3aa603a8a23207d7aa177f3fa7cca5ff34
                                 </geometry>
                               </visual>
@@ -242,5 +355,9 @@
                                 <origin xyz="0 0 0" rpy="0 0 -1.5"/>
                                   <geometry>
+<<<<<<< HEAD
+                                    <mesh filename="package://insect_description/meshes/leg_v1.dae" />
+=======
                                     <mesh filename="package://insect_description/meshes/leg_v1.dae"/>
+>>>>>>> 91e1ca3aa603a8a23207d7aa177f3fa7cca5ff34
                                   </geometry>
                                 </collision>
@@ -248,5 +365,9 @@
                                   <origin xyz="0 0 0" rpy="0 0 -1.5"/>
                                   <geometry>
+<<<<<<< HEAD
+                                    <mesh filename="package://insect_description/meshes/leg_v1.dae" />
+=======
                                     <mesh filename="package://insect_description/meshes/leg_v1.dae"/>
+>>>>>>> 91e1ca3aa603a8a23207d7aa177f3fa7cca5ff34
                                   </geometry>
                                 </visual>
@@ -257,5 +378,9 @@
                                   <origin xyz="0 0 0" rpy="0 0 1.5"/>
                                     <geometry>
+<<<<<<< HEAD
+                                      <mesh filename="package://insect_description/meshes/leg_v1.dae" />
+=======
                                       <mesh filename="package://insect_description/meshes/leg_v1.dae"/>
+>>>>>>> 91e1ca3aa603a8a23207d7aa177f3fa7cca5ff34
                                     </geometry>
                                   </collision>
@@ -263,5 +388,9 @@
                                     <origin xyz="0 0 0" rpy="0 0 1.5"/>
                                     <geometry>
+<<<<<<< HEAD
+                                      <mesh filename="package://insect_description/meshes/leg_v1.dae" />
+=======
                                       <mesh filename="package://insect_description/meshes/leg_v1.dae"/>
+>>>>>>> 91e1ca3aa603a8a23207d7aa177f3fa7cca5ff34
                                     </geometry>
                                   </visual>
@@ -272,5 +401,9 @@
                                     <origin xyz="0 0 0" rpy="0 0 1.5"/>
                                       <geometry>
+<<<<<<< HEAD
+                                        <mesh filename="package://insect_description/meshes/leg_v1.dae" />
+=======
                                         <mesh filename="package://insect_description/meshes/leg_v1.dae"/>
+>>>>>>> 91e1ca3aa603a8a23207d7aa177f3fa7cca5ff34
                                       </geometry>
                                     </collision>
@@ -278,9 +411,13 @@
                                       <origin xyz="0 0 0" rpy="0 0 1.5"/>
                                       <geometry>
+<<<<<<< HEAD
+                                        <mesh filename="package://insect_description/meshes/leg_v1.dae" />
+=======
                                         <mesh filename="package://insect_description/meshes/leg_v1.dae"/>
+>>>>>>> 91e1ca3aa603a8a23207d7aa177f3fa7cca5ff34
                                       </geometry>
                                     </visual>
                                     <xacro:default_inertial mass="0.4"/>
-                                  </link>
+                                  </link-->
 <!--############################################################################################################################-->
                                   <!--link name="hokuyo_link">
@@ -292,5 +429,9 @@
                                       </collision>     <origin xyz="0 0 0" rpy="0 0 0"/>
                                           <geometry-->
+<<<<<<< HEAD
+                                              <!--mesh filename="package://insect/meshes/hokuyo.dae"/-->
+=======
                                               <!--mesh filename="package://://insect/meshes/hokuyo.dae"/-->
+>>>>>>> 91e1ca3aa603a8a23207d7aa177f3fa7cca5ff34
                                               <!--mesh filename="package://insect_description/meshes/hokuyo.dae"/>
                                           </geometry>
@@ -298,5 +439,9 @@
                                           <origin xyz="0 0 0" rpy="0 0 0"/>
                                           <geometry-->
+<<<<<<< HEAD
+                                              <!--mesh filename="package://insect/meshes/hokuyo.dae"/-->
+=======
                                               <!--mesh filename="package://://insect/meshes/hokuyo.dae"/-->
+>>>>>>> 91e1ca3aa603a8a23207d7aa177f3fa7cca5ff34
                                               <!--mesh filename="package://insect_description/meshes/hokuyo.dae"/>
                                           </geometry>
@@ -312,9 +457,13 @@
 <xacro:property name="joint_lower_limit" value="-${3.14}"/>
 <xacro:property name="joint_upper_limit" value="${3.14}"/>
-<xacro:property name="joint_effort" value="6.0"/>
+<xacro:property name="joint_effort" value="2.0"/>
 <xacro:property name="joint_velocity" value="0.524"/>
 <!--######################################################################################################################################-->
 <!--joint name="hokuyo_joint" type="fixed">
+<<<<<<< HEAD
+    <origin xyz="0.04 0 0.08" rpy="0 0 0"/>
+=======
     <origin xyz="0 0 0.08" rpy="0 0 0"/>
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