Commit message: modified urdf

File: insect_description/urdf/insect.urdf.xacro (robot description, xacro)
@@ -1,3 +1,3 @@
-<?xml version="1.0" encoding="UTF-8"?>
+<?xml version='1.0'?>
 <robot name="insect" xmlns:xacro="http://www.ros.org/wiki/xacro">
 <!--##################################################################################################################################-->
@@ -7,5 +7,4 @@
 <xacro:macro name="default_inertial" params="mass">
    <inertial>
-     <origin xyz="0.0 0.0 0.0" rpy="0.0 0.0 0.0" />
      <mass value="${mass}" />
      <inertia ixx="1.0" ixy="0.0" ixz="0.0" iyy="1.0" iyz="0.0" izz="1.0" />
@@ -18,9 +17,5 @@
   <origin xyz="0 0 0" rpy="0 0 0"/>
   <geometry>
-<<<<<<< HEAD
-    <mesh filename="package://insect_description/meshes/torso_v1.dae" />
-=======
     <mesh filename="package://insect_description/meshes/torso_v1.dae"/>
->>>>>>> 91e1ca3aa603a8a23207d7aa177f3fa7cca5ff34
   </geometry>
 </collision>
@@ -28,9 +23,5 @@
   <origin xyz="0 0 0" rpy="0 0 0"/>
   <geometry>
-<<<<<<< HEAD
-    <mesh filename="package://insect_description/meshes/torso_v1.dae" />
-=======
     <mesh filename="package://insect_description/meshes/torso_v1.dae"/>
->>>>>>> 91e1ca3aa603a8a23207d7aa177f3fa7cca5ff34
   </geometry>
 </visual>
@@ -54,34 +45,22 @@
   <link name= "l_f_motor">
     <collision name="collision">
-      <origin xyz="0 0 0" rpy="0 -0.5 -1.5"/>
+      <origin xyz="0 0 0" rpy="0 0 0"/>
         <geometry>
-<<<<<<< HEAD
-          <mesh filename="package://insect_description/meshes/motor_v1.dae" />
-=======
           <mesh filename="package://insect_description/meshes/motor_v1.dae"/>
->>>>>>> 91e1ca3aa603a8a23207d7aa177f3fa7cca5ff34
         </geometry>
       </collision>
       <visual name="visual">
-        <origin xyz="0 0 0" rpy="0 -0.5 -1.4"/>
+        <origin xyz="0 0 0" rpy="0 0 0"/>
         <geometry>
-<<<<<<< HEAD
-          <mesh filename="package://insect_description/meshes/motor_v1.dae" />
-=======
           <mesh filename="package://insect_description/meshes/motor_v1.dae"/>
->>>>>>> 91e1ca3aa603a8a23207d7aa177f3fa7cca5ff34
         </geometry>
       </visual>
       <xacro:default_inertial mass="0.2"/>
     </link>
-    <!--link name= "r_f_motor">
+    <link name= "r_f_motor">
       <collision name="collision">
         <origin xyz="0 0 0" rpy="0 -0.5 1.5"/>
           <geometry>
-<<<<<<< HEAD
-            <mesh filename="package://insect_description/meshes/motor_v1.dae" />
-=======
             <mesh filename="package://insect_description/meshes/motor_v1.dae"/>
->>>>>>> 91e1ca3aa603a8a23207d7aa177f3fa7cca5ff34
           </geometry>
         </collision>
@@ -89,9 +68,5 @@
           <origin xyz="0 0 0" rpy="0 -0.5 1.5"/>
           <geometry>
-<<<<<<< HEAD
-            <mesh filename="package://insect_description/meshes/motor_v1.dae" />
-=======
             <mesh filename="package://insect_description/meshes/motor_v1.dae"/>
->>>>>>> 91e1ca3aa603a8a23207d7aa177f3fa7cca5ff34
           </geometry>
         </visual>
@@ -102,9 +77,5 @@
           <origin xyz="0 0 0" rpy="0 -0.5 -1.5"/>
             <geometry>
-<<<<<<< HEAD
-              <mesh filename="package://insect_description/meshes/motor_v1.dae" />
-=======
               <mesh filename="package://insect_description/meshes/motor_v1.dae"/>
->>>>>>> 91e1ca3aa603a8a23207d7aa177f3fa7cca5ff34
             </geometry>
           </collision>
@@ -112,9 +83,5 @@
             <origin xyz="0 0 0" rpy="0 -0.5 -1.5"/>
             <geometry>
-<<<<<<< HEAD
-              <mesh filename="package://insect_description/meshes/motor_v1.dae" />
-=======
               <mesh filename="package://insect_description/meshes/motor_v1.dae"/>
->>>>>>> 91e1ca3aa603a8a23207d7aa177f3fa7cca5ff34
             </geometry>
           </visual>
@@ -125,9 +92,5 @@
             <origin xyz="0 0 0" rpy="0 -0.5 1.5"/>
               <geometry>
-<<<<<<< HEAD
-                <mesh filename="package://insect_description/meshes/motor_v1.dae" />
-=======
                 <mesh filename="package://insect_description/meshes/motor_v1.dae"/>
->>>>>>> 91e1ca3aa603a8a23207d7aa177f3fa7cca5ff34
               </geometry>
             </collision>
@@ -135,45 +98,29 @@
               <origin xyz="0 0 0" rpy="0 -0.5 1.5"/>
               <geometry>
-<<<<<<< HEAD
-                <mesh filename="package://insect_description/meshes/motor_v1.dae" />
-=======
                 <mesh filename="package://insect_description/meshes/motor_v1.dae"/>
->>>>>>> 91e1ca3aa603a8a23207d7aa177f3fa7cca5ff34
               </geometry>
             </visual>
             <xacro:default_inertial mass="0.2"/>
-          </link-->
+          </link>
           <link name= "l_f_hip">
             <collision name="collision">
-              <origin xyz="0 0 0" rpy="0 -0.5 -1.5"/>
+              <origin xyz="0 0 0" rpy="0 0 0"/>
                 <geometry>
-<<<<<<< HEAD
-                  <mesh filename="package://insect_description/meshes/hip_v1.dae" />
-=======
                   <mesh filename="package://insect_description/meshes/hip_v1.dae"/>
->>>>>>> 91e1ca3aa603a8a23207d7aa177f3fa7cca5ff34
                 </geometry>
               </collision>
               <visual name="visual">
-                <origin xyz="0 0 0" rpy="0 -0.5 -1.5"/>
+                <origin xyz="0 0 0" rpy="0 0 0"/>
                 <geometry>
-<<<<<<< HEAD
-                  <mesh filename="package://insect_description/meshes/hip_v1.dae" />
-=======
                   <mesh filename="package://insect_description/meshes/hip_v1.dae"/>
->>>>>>> 91e1ca3aa603a8a23207d7aa177f3fa7cca5ff34
                 </geometry>
               </visual>
               <xacro:default_inertial mass="0.4"/>
             </link>
-            <!--link name= "r_f_hip">
+            <link name= "r_f_hip">
               <collision name="collision">
                 <origin xyz="0 0 0" rpy="0 -0.5 1.5"/>
                   <geometry>
-<<<<<<< HEAD
-                    <mesh filename="package://insect_description/meshes/hip_v1.dae" />
-=======
                     <mesh filename="package://insect_description/meshes/hip_v1.dae"/>
->>>>>>> 91e1ca3aa603a8a23207d7aa177f3fa7cca5ff34
                   </geometry>
                 </collision>
@@ -181,9 +128,5 @@
                   <origin xyz="0 0 0" rpy="0 -0.5 1.5"/>
                   <geometry>
-<<<<<<< HEAD
-                    <mesh filename="package://insect_description/meshes/hip_v1.dae" />
-=======
                     <mesh filename="package://insect_description/meshes/hip_v1.dae"/>
->>>>>>> 91e1ca3aa603a8a23207d7aa177f3fa7cca5ff34
                   </geometry>
                 </visual>
@@ -194,9 +137,5 @@
                   <origin xyz="0 0 0" rpy="0 -0.5 -1.5"/>
                     <geometry>
-<<<<<<< HEAD
-                      <mesh filename="package://insect_description/meshes/hip_v1.dae" />
-=======
                       <mesh filename="package://insect_description/meshes/hip_v1.dae"/>
->>>>>>> 91e1ca3aa603a8a23207d7aa177f3fa7cca5ff34
                     </geometry>
                   </collision>
@@ -204,9 +143,5 @@
                     <origin xyz="0 0 0" rpy="0 -0.5 -1.5"/>
                     <geometry>
-<<<<<<< HEAD
-                      <mesh filename="package://insect_description/meshes/hip_v1.dae" />
-=======
                       <mesh filename="package://insect_description/meshes/hip_v1.dae"/>
->>>>>>> 91e1ca3aa603a8a23207d7aa177f3fa7cca5ff34
                     </geometry>
                   </visual>
@@ -217,9 +152,5 @@
                     <origin xyz="0 0 0" rpy="0 -0.5 1.5"/>
                       <geometry>
-<<<<<<< HEAD
-                        <mesh filename="package://insect_description/meshes/hip_v1.dae" />
-=======
                         <mesh filename="package://insect_description/meshes/hip_v1.dae"/>
->>>>>>> 91e1ca3aa603a8a23207d7aa177f3fa7cca5ff34
                       </geometry>
                     </collision>
@@ -227,22 +158,14 @@
                       <origin xyz="0 0 0" rpy="0 -0.5 1.5"/>
                       <geometry>
-<<<<<<< HEAD
-                        <mesh filename="package://insect_description/meshes/hip_v1.dae" />
-=======
                         <mesh filename="package://insect_description/meshes/hip_v1.dae"/>
->>>>>>> 91e1ca3aa603a8a23207d7aa177f3fa7cca5ff34
                       </geometry>
                     </visual>
                     <xacro:default_inertial mass="0.4"/>
                   </link>
-                  <link name= "l_f_h_motor">
+                  <!--link name= "l_f_h_motor">
                     <collision name="collision">
                       <origin xyz="0 0 0" rpy="0 -3.4 -1.5"/>
                         <geometry>
-<<<<<<< HEAD
-                          <mesh filename="package://insect_description/meshes/motor_h_v1.dae" />
-=======
                           <mesh filename="package://insect_description/meshes/motor_h_v1.dae"/>
->>>>>>> 91e1ca3aa603a8a23207d7aa177f3fa7cca5ff34
                         </geometry>
                       </collision>
@@ -250,22 +173,14 @@
                         <origin xyz="0 0 0" rpy="0 -3.4 -1.5"/>
                         <geometry>
-<<<<<<< HEAD
-                          <mesh filename="package://insect_description/meshes/motor_h_v1.dae" />
-=======
                           <mesh filename="package://insect_description/meshes/motor_h_v1.dae"/>
->>>>>>> 91e1ca3aa603a8a23207d7aa177f3fa7cca5ff34
                         </geometry>
                       </visual>
                       <xacro:default_inertial mass="0.2"/>
-                    </link>
+                    </link-->
                     <link name= "r_f_h_motor">
                       <collision name="collision">
                         <origin xyz="0 0 0" rpy="0 -3.4 -1.5"/>
                           <geometry>
-<<<<<<< HEAD
-                            <mesh filename="package://insect_description/meshes/motor_h_v1.dae" />
-=======
                             <mesh filename="package://insect_description/meshes/motor_h_v1.dae"/>
->>>>>>> 91e1ca3aa603a8a23207d7aa177f3fa7cca5ff34
                           </geometry>
                         </collision>
@@ -273,9 +188,5 @@
                           <origin xyz="0 0 0" rpy="0 -3.4 1.5"/>
                           <geometry>
-<<<<<<< HEAD
-                            <mesh filename="package://insect_description/meshes/motor_h_v1.dae" />
-=======
                             <mesh filename="package://insect_description/meshes/motor_h_v1.dae"/>
->>>>>>> 91e1ca3aa603a8a23207d7aa177f3fa7cca5ff34
                           </geometry>
                         </visual>
@@ -286,9 +197,5 @@
                           <origin xyz="0 0 0" rpy="0 -3.4 -1.5"/>
                             <geometry>
-<<<<<<< HEAD
-                              <mesh filename="package://insect_description/meshes/motor_h_v1.dae" />
-=======
                               <mesh filename="package://insect_description/meshes/motor_h_v1.dae"/>
->>>>>>> 91e1ca3aa603a8a23207d7aa177f3fa7cca5ff34
                             </geometry>
                           </collision>
@@ -296,9 +203,5 @@
                             <origin xyz="0 0 0" rpy="0 -3.4 -1.5"/>
                             <geometry>
-<<<<<<< HEAD
-                              <mesh filename="package://insect_description/meshes/motor_h_v1.dae" />
-=======
                               <mesh filename="package://insect_description/meshes/motor_h_v1.dae"/>
->>>>>>> 91e1ca3aa603a8a23207d7aa177f3fa7cca5ff34
                             </geometry>
                           </visual>
@@ -309,9 +212,5 @@
                             <origin xyz="0 0 0" rpy="0 -3.4 -1.5"/>
                               <geometry>
-<<<<<<< HEAD
-                                <mesh filename="package://insect_description/meshes/motor_h_v1.dae" />
-=======
                                 <mesh filename="package://insect_description/meshes/motor_h_v1.dae"/>
->>>>>>> 91e1ca3aa603a8a23207d7aa177f3fa7cca5ff34
                               </geometry>
                             </collision>
@@ -319,22 +218,14 @@
                               <origin xyz="0 0 0" rpy="0 -3.4 1.5"/>
                               <geometry>
-<<<<<<< HEAD
-                                <mesh filename="package://insect_description/meshes/motor_h_v1.dae" />
-=======
                                 <mesh filename="package://insect_description/meshes/motor_h_v1.dae"/>
->>>>>>> 91e1ca3aa603a8a23207d7aa177f3fa7cca5ff34
                               </geometry>
                             </visual>
                             <xacro:default_inertial mass="0.2"/>
                           </link>
-                          <link name= "l_f_leg">
+                          <!--link name= "l_f_le1.57g">
                             <collision name="collision">
                               <origin xyz="0 0 0" rpy="0 0 -1.5"/>
                                 <geometry>
-<<<<<<< HEAD
-                                  <mesh filename="package://insect_description/meshes/leg_v1.dae" />
-=======
                                   <mesh filename="package://insect_description/meshes/leg_v1.dae"/>
->>>>>>> 91e1ca3aa603a8a23207d7aa177f3fa7cca5ff34
                                 </geometry>
                               </collision>
@@ -342,22 +233,14 @@
                                 <origin xyz="0 0 0" rpy="0 0 -1.5"/>
                                 <geometry>
-<<<<<<< HEAD
-                                  <mesh filename="package://insect_description/meshes/leg_v1.dae" />
-=======
                                   <mesh filename="package://insect_description/meshes/leg_v1.dae"/>
->>>>>>> 91e1ca3aa603a8a23207d7aa177f3fa7cca5ff34
                                 </geometry>
                               </visual>
                               <xacro:default_inertial mass="0.4"/>
-                            </link>
+                            </link-->
                             <link name= "l_b_leg">
                               <collision name="collision">
                                 <origin xyz="0 0 0" rpy="0 0 -1.5"/>
                                   <geometry>
-<<<<<<< HEAD
-                                    <mesh filename="package://insect_description/meshes/leg_v1.dae" />
-=======
                                     <mesh filename="package://insect_description/meshes/leg_v1.dae"/>
->>>>>>> 91e1ca3aa603a8a23207d7aa177f3fa7cca5ff34
                                   </geometry>
                                 </collision>
@@ -365,9 +248,5 @@
                                   <origin xyz="0 0 0" rpy="0 0 -1.5"/>
                                   <geometry>
-<<<<<<< HEAD
-                                    <mesh filename="package://insect_description/meshes/leg_v1.dae" />
-=======
                                     <mesh filename="package://insect_description/meshes/leg_v1.dae"/>
->>>>>>> 91e1ca3aa603a8a23207d7aa177f3fa7cca5ff34
                                   </geometry>
                                 </visual>
@@ -378,9 +257,5 @@
                                   <origin xyz="0 0 0" rpy="0 0 1.5"/>
                                     <geometry>
-<<<<<<< HEAD
-                                      <mesh filename="package://insect_description/meshes/leg_v1.dae" />
-=======
                                       <mesh filename="package://insect_description/meshes/leg_v1.dae"/>
->>>>>>> 91e1ca3aa603a8a23207d7aa177f3fa7cca5ff34
                                     </geometry>
                                   </collision>
@@ -388,9 +263,5 @@
                                     <origin xyz="0 0 0" rpy="0 0 1.5"/>
                                     <geometry>
-<<<<<<< HEAD
-                                      <mesh filename="package://insect_description/meshes/leg_v1.dae" />
-=======
                                       <mesh filename="package://insect_description/meshes/leg_v1.dae"/>
->>>>>>> 91e1ca3aa603a8a23207d7aa177f3fa7cca5ff34
                                     </geometry>
                                   </visual>
@@ -401,9 +272,5 @@
                                     <origin xyz="0 0 0" rpy="0 0 1.5"/>
                                       <geometry>
-<<<<<<< HEAD
-                                        <mesh filename="package://insect_description/meshes/leg_v1.dae" />
-=======
                                         <mesh filename="package://insect_description/meshes/leg_v1.dae"/>
->>>>>>> 91e1ca3aa603a8a23207d7aa177f3fa7cca5ff34
                                       </geometry>
                                     </collision>
@@ -411,13 +278,9 @@
                                       <origin xyz="0 0 0" rpy="0 0 1.5"/>
                                       <geometry>
-<<<<<<< HEAD
-                                        <mesh filename="package://insect_description/meshes/leg_v1.dae" />
-=======
                                         <mesh filename="package://insect_description/meshes/leg_v1.dae"/>
->>>>>>> 91e1ca3aa603a8a23207d7aa177f3fa7cca5ff34
                                       </geometry>
                                     </visual>
                                     <xacro:default_inertial mass="0.4"/>
-                                  </link-->
+                                  </link>
 <!--############################################################################################################################-->
                                   <!--link name="hokuyo_link">
@@ -429,9 +292,5 @@
                                       </collision>     <origin xyz="0 0 0" rpy="0 0 0"/>
                                           <geometry-->
-<<<<<<< HEAD
-                                              <!--mesh filename="package://insect/meshes/hokuyo.dae"/-->
-=======
                                               <!--mesh filename="package://://insect/meshes/hokuyo.dae"/-->
->>>>>>> 91e1ca3aa603a8a23207d7aa177f3fa7cca5ff34
                                               <!--mesh filename="package://insect_description/meshes/hokuyo.dae"/>
                                           </geometry>
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