Commit message: joint parameter modified

File: insect_description/urdf/insect.urdf.xacro (robot description, xacro)
@@ -60,5 +60,5 @@
     <link name= "r_f_motor">
       <collision name="collision">
-        <origin xyz="0 0 0" rpy="0 -0.5 1.5"/>
+        <origin xyz="0 0 0" rpy="0 0 0"/>
           <geometry>
             <mesh filename="package://insect_description/meshes/motor_v1.dae"/>
@@ -66,5 +66,5 @@
         </collision>
         <visual name="visual">
-          <origin xyz="0 0 0" rpy="0 -0.5 1.5"/>
+          <origin xyz="0 0 0" rpy="0 0 0"/>
           <geometry>
             <mesh filename="package://insect_description/meshes/motor_v1.dae"/>
@@ -75,5 +75,5 @@
       <link name= "l_b_motor">
         <collision name="collision">
-          <origin xyz="0 0 0" rpy="0 -0.5 -1.5"/>
+          <origin xyz="0 0 0" rpy="0 0 0"/>
             <geometry>
               <mesh filename="package://insect_description/meshes/motor_v1.dae"/>
@@ -81,5 +81,5 @@
           </collision>
           <visual name="visual">
-            <origin xyz="0 0 0" rpy="0 -0.5 -1.5"/>
+            <origin xyz="0 0 0" rpy="0 0 0"/>
             <geometry>
               <mesh filename="package://insect_description/meshes/motor_v1.dae"/>
@@ -90,5 +90,5 @@
         <link name= "r_b_motor">
           <collision name="collision">
-            <origin xyz="0 0 0" rpy="0 -0.5 1.5"/>
+            <origin xyz="0 0 0" rpy="0 0 0"/>
               <geometry>
                 <mesh filename="package://insect_description/meshes/motor_v1.dae"/>
@@ -96,5 +96,5 @@
             </collision>
             <visual name="visual">
-              <origin xyz="0 0 0" rpy="0 -0.5 1.5"/>
+              <origin xyz="0 0 0" rpy="0 0 0"/>
               <geometry>
                 <mesh filename="package://insect_description/meshes/motor_v1.dae"/>
@@ -120,5 +120,5 @@
             <link name= "r_f_hip">
               <collision name="collision">
-                <origin xyz="0 0 0" rpy="0 -0.5 1.5"/>
+                <origin xyz="0 0 0" rpy="0 0 0"/>
                   <geometry>
                     <mesh filename="package://insect_description/meshes/hip_v1.dae"/>
@@ -126,5 +126,5 @@
                 </collision>
                 <visual name="visual">
-                  <origin xyz="0 0 0" rpy="0 -0.5 1.5"/>
+                  <origin xyz="0 0 0" rpy="0 0 0"/>
                   <geometry>
                     <mesh filename="package://insect_description/meshes/hip_v1.dae"/>
@@ -135,5 +135,5 @@
               <link name= "l_b_hip">
                 <collision name="collision">
-                  <origin xyz="0 0 0" rpy="0 -0.5 -1.5"/>
+                  <origin xyz="0 0 0" rpy="0 0 0"/>
                     <geometry>
                       <mesh filename="package://insect_description/meshes/hip_v1.dae"/>
@@ -141,5 +141,5 @@
                   </collision>
                   <visual name="visual">
-                    <origin xyz="0 0 0" rpy="0 -0.5 -1.5"/>
+                    <origin xyz="0 0 0" rpy="0 0 0"/>
                     <geometry>
                       <mesh filename="package://insect_description/meshes/hip_v1.dae"/>
@@ -150,5 +150,5 @@
                 <link name= "r_b_hip">
                   <collision name="collision">
-                    <origin xyz="0 0 0" rpy="0 -0.5 1.5"/>
+                    <origin xyz="0 0 0" rpy="0 0 0"/>
                       <geometry>
                         <mesh filename="package://insect_description/meshes/hip_v1.dae"/>
@@ -156,5 +156,5 @@
                     </collision>
                     <visual name="visual">
-                      <origin xyz="0 0 0" rpy="0 -0.5 1.5"/>
+                      <origin xyz="0 0 0" rpy="0 0 0"/>
                       <geometry>
                         <mesh filename="package://insect_description/meshes/hip_v1.dae"/>
@@ -163,7 +163,7 @@
                     <xacro:default_inertial mass="0.4"/>
                   </link>
-                  <!--link name= "l_f_h_motor">
+                  <link name= "l_f_h_motor">
                     <collision name="collision">
-                      <origin xyz="0 0 0" rpy="0 -3.4 -1.5"/>
+                      <origin xyz="0 0 0" rpy="0 0 0"/>
                         <geometry>
                           <mesh filename="package://insect_description/meshes/motor_h_v1.dae"/>
@@ -171,5 +171,5 @@
                       </collision>
                       <visual name="visual">
-                        <origin xyz="0 0 0" rpy="0 -3.4 -1.5"/>
+                        <origin xyz="0 0 0" rpy="0 0 0"/>
                         <geometry>
                           <mesh filename="package://insect_description/meshes/motor_h_v1.dae"/>
@@ -177,8 +177,8 @@
                       </visual>
                       <xacro:default_inertial mass="0.2"/>
-                    </link-->
+                    </link>
                     <link name= "r_f_h_motor">
                       <collision name="collision">
-                        <origin xyz="0 0 0" rpy="0 -3.4 -1.5"/>
+                        <origin xyz="0 0 0" rpy="0 0 0"/>
                           <geometry>
                             <mesh filename="package://insect_description/meshes/motor_h_v1.dae"/>
@@ -186,5 +186,5 @@
                         </collision>
                         <visual name="visual">
-                          <origin xyz="0 0 0" rpy="0 -3.4 1.5"/>
+                          <origin xyz="0 0 0" rpy="0 0 0"/>
                           <geometry>
                             <mesh filename="package://insect_description/meshes/motor_h_v1.dae"/>
@@ -195,5 +195,5 @@
                       <link name= "l_b_h_motor">
                         <collision name="collision">
-                          <origin xyz="0 0 0" rpy="0 -3.4 -1.5"/>
+                          <origin xyz="0 0 0" rpy="0 0 0"/>
                             <geometry>
                               <mesh filename="package://insect_description/meshes/motor_h_v1.dae"/>
@@ -201,5 +201,5 @@
                           </collision>
                           <visual name="visual">
-                            <origin xyz="0 0 0" rpy="0 -3.4 -1.5"/>
+                            <origin xyz="0 0 0" rpy="0 0 0"/>
                             <geometry>
                               <mesh filename="package://insect_description/meshes/motor_h_v1.dae"/>
@@ -210,5 +210,5 @@
                         <link name= "r_b_h_motor">
                           <collision name="collision">
-                            <origin xyz="0 0 0" rpy="0 -3.4 -1.5"/>
+                            <origin xyz="0 0 0" rpy="0 0 0"/>
                               <geometry>
                                 <mesh filename="package://insect_description/meshes/motor_h_v1.dae"/>
@@ -216,5 +216,5 @@
                             </collision>
                             <visual name="visual">
-                              <origin xyz="0 0 0" rpy="0 -3.4 1.5"/>
+                              <origin xyz="0 0 0" rpy="0 0 0"/>
                               <geometry>
                                 <mesh filename="package://insect_description/meshes/motor_h_v1.dae"/>
@@ -223,7 +223,7 @@
                             <xacro:default_inertial mass="0.2"/>
                           </link>
-                          <!--link name= "l_f_le1.57g">
+                          <link name= "l_f_leg">
                             <collision name="collision">
-                              <origin xyz="0 0 0" rpy="0 0 -1.5"/>
+                              <origin xyz="0 0 0" rpy="0 0 0"/>
                                 <geometry>
                                   <mesh filename="package://insect_description/meshes/leg_v1.dae"/>
@@ -231,5 +231,5 @@
                               </collision>
                               <visual name="visual">
-                                <origin xyz="0 0 0" rpy="0 0 -1.5"/>
+                                <origin xyz="0 0 0" rpy="0 0 0"/>
                                 <geometry>
                                   <mesh filename="package://insect_description/meshes/leg_v1.dae"/>
@@ -237,8 +237,8 @@
                               </visual>
                               <xacro:default_inertial mass="0.4"/>
-                            </link-->
+                            </link>
                             <link name= "l_b_leg">
                               <collision name="collision">
-                                <origin xyz="0 0 0" rpy="0 0 -1.5"/>
+                                <origin xyz="0 0 0" rpy="0 0 0"/>
                                   <geometry>
                                     <mesh filename="package://insect_description/meshes/leg_v1.dae"/>
@@ -246,5 +246,5 @@
                                 </collision>
                                 <visual name="visual">
-                                  <origin xyz="0 0 0" rpy="0 0 -1.5"/>
+                                  <origin xyz="0 0 0" rpy="0 0 0"/>
                                   <geometry>
                                     <mesh filename="package://insect_description/meshes/leg_v1.dae"/>
@@ -255,5 +255,5 @@
                               <link name= "r_f_leg">
                                 <collision name="collision">
-                                  <origin xyz="0 0 0" rpy="0 0 1.5"/>
+                                  <origin xyz="0 0 0" rpy="0 0 0"/>
                                     <geometry>
                                       <mesh filename="package://insect_description/meshes/leg_v1.dae"/>
@@ -261,5 +261,5 @@
                                   </collision>
                                   <visual name="visual">
-                                    <origin xyz="0 0 0" rpy="0 0 1.5"/>
+                                    <origin xyz="0 0 0" rpy="0 0 0"/>
                                     <geometry>
                                       <mesh filename="package://insect_description/meshes/leg_v1.dae"/>
@@ -270,5 +270,5 @@
                                 <link name= "r_b_leg">
                                   <collision name="collision">
-                                    <origin xyz="0 0 0" rpy="0 0 1.5"/>
+                                    <origin xyz="0 0 0" rpy="0 0 0"/>
                                       <geometry>
                                         <mesh filename="package://insect_description/meshes/leg_v1.dae"/>
@@ -276,5 +276,5 @@
                                     </collision>
                                     <visual name="visual">
-                                      <origin xyz="0 0 0" rpy="0 0 1.5"/>
+                                      <origin xyz="0 0 0" rpy="0 0 0"/>
                                       <geometry>
                                         <mesh filename="package://insect_description/meshes/leg_v1.dae"/>
@@ -284,5 +284,5 @@
                                   </link>
 <!--############################################################################################################################-->
-                                  <!--link name="hokuyo_link">
+                                  <link name="hokuyo_link">
                                       <collision>
                                           <origin xyz="0 0 0" rpy="0 0 0"/>
@@ -291,13 +291,11 @@
                                           </geometry>
                                       </collision>     <origin xyz="0 0 0" rpy="0 0 0"/>
-                                          <geometry-->
-                                              <!--mesh filename="package://://insect/meshes/hokuyo.dae"/-->
-                                              <!--mesh filename="package://insect_description/meshes/hokuyo.dae"/>
+                                          <geometry>
+                                              <mesh filename="package://insect_description/meshes/hokuyo.dae"/>
                                           </geometry>
                                       <visual>
                                           <origin xyz="0 0 0" rpy="0 0 0"/>
-                                          <geometry-->
-                                              <!--mesh filename="package://://insect/meshes/hokuyo.dae"/-->
-                                              <!--mesh filename="package://insect_description/meshes/hokuyo.dae"/>
+                                          <geometry>
+                                              <mesh filename="package://insect_description/meshes/hokuyo.dae"/>
                                           </geometry>
                                       </visual>
@@ -307,5 +305,5 @@
                                           <inertia ixx="1e-6" ixy="0" ixz="0" iyy="1e-6" iyz="0" izz="1e-6" />
                                       </inertial>
-                                  </link-->
+                                  </link>
 <!--#########################################################################################################################################-->
 <!-- Joint properties -->
@@ -316,11 +314,11 @@
 <xacro:property name="pi" value="3.1415926535897931"/>
 <!--######################################################################################################################################-->
-<!--joint name="hokuyo_joint" type="fixed">
+<joint name="hokuyo_joint" type="fixed">
     <origin xyz="0 0 0.08" rpy="0 0 0"/>
     <parent link="torso_base"/>
     <child link="hokuyo_link"/>
-</joint-->
+</joint>
 <joint name="world_joint"  type="fixed">
-  <origin xyz="0 0 0.30" rpy="0 0 0" />
+  <origin xyz="0 0 0.50" rpy="0 0 0" />
   <parent link="world"/>
   <child link="torso_base"/>
@@ -341,5 +339,5 @@
 </joint>
 <joint name="r_f_motor_joint"  type="fixed">
-  <origin xyz="0.048 -0.09 -0.08" rpy="0 0 0" />
+  <origin xyz="0.048 -0.09 -0.08" rpy="0 -${pi/6} ${pi/2}" />
   <parent link="torso_base"/>
   <child link="r_f_motor"/>
@@ -347,5 +345,5 @@
 </joint>
 <joint name="l_b_motor_joint"  type="fixed">
-  <origin xyz="-0.2 0.08 -0.08" rpy="0 0 0" />
+  <origin xyz="-0.2 0.08 -0.08" rpy="0 -${pi/6} -${pi/2}" />
   <parent link="torso_base"/>
   <child link="l_b_motor"/>
@@ -353,5 +351,5 @@
 </joint>
 <joint name="r_b_motor_joint"  type="fixed">
-  <origin xyz="-0.2 -0.09 -0.08" rpy="0 0 0" />
+  <origin xyz="-0.2 -0.09 -0.08" rpy="0 -${pi/6} ${pi/2}"/>
   <parent link="torso_base"/>
   <child link="r_b_motor"/>
@@ -359,37 +357,39 @@
 </joint>
 <joint name="l_f_hip_joint"  type="revolute">
-  <origin xyz=" 0.048 0.09 -0.08" rpy="0 0 ${pi}" />
+  <origin xyz=" -0.04 -0.00005 -0.054" rpy="0 0 0" />
   <parent link="l_f_motor"/>
   <child link="l_f_hip"/>
   <limit lower="${joint_lower_limit}" upper="${joint_upper_limit}" effort="${joint_effort}" velocity="${joint_velocity}"/>
-  <axis xyz="0 0 1" rpy="0 0 0"/>
-</joint>
-<joint name="r_f_hip_joint"  type="fixed">
-  <origin xyz="0.006 -0.01 -0.067" rpy="0 0 0" />
+  <axis xyz="0 0 1"/>
+</joint>
+  <joint name="r_f_hip_joint"  type="revolute">
+  <origin xyz="-0.04 0.00005 -0.054" rpy="0 0 0" />
   <parent link="r_f_motor"/>
   <child link="r_f_hip"/>
-  <!--limit lower="${joint_lower_limit}" upper="${joint_upper_limit}" effort="${joint_effort}" velocity="${joint_velocity}"/-->
-  <axis xyz="0 0 1" rpy="0 0 0"/>
-</joint>
-<joint name="l_b_hip_joint"  type="fixed">
-  <origin xyz="0.006 0.01 -0.067" rpy="0 0 0" />
+  <limit lower="${joint_lower_limit}" upper="${joint_upper_limit}" effort="${joint_effort}" velocity="${joint_velocity}"/>
+  <axis xyz="0 0 1" rpy="0 0 0"/>
+</joint>
+ <joint name="l_b_hip_joint"  type="revolute">
+  <origin xyz="-0.04 0.003 -0.054" rpy="0 0 0" />
   <parent link="l_b_motor"/>
   <child link="l_b_hip"/>
   <axis xyz="0 0 1" rpy="0 0 0"/>
-</joint>
-<joint name="r_b_hip_joint"  type="fixed">
-  <origin xyz="-0.006 -0.01 -0.067" rpy="0 0 0" />
+  <limit lower="${joint_lower_limit}" upper="${joint_upper_limit}" effort="${joint_effort}" velocity="${joint_velocity}"/>
+</joint>
+ <joint name="r_b_hip_joint"  type="revolute">
+  <origin xyz="-0.04 0.003 -0.054" rpy="0 0 0" />
   <parent link="r_b_motor"/>
   <child link="r_b_hip"/>
-  <axis xyz="0 0 1" rpy="0 0 0"/>
-</joint>
-<!--joint name="l_f_h_motor_joint"  type="fixed">
-  <origin xyz="-0.014 0.163 0.088" rpy="0 0 0" />
+  <limit lower="${joint_lower_limit}" upper="${joint_upper_limit}" effort="${joint_effort}" velocity="${joint_velocity}"/>
+  <axis xyz="0 0 1" rpy="0 0 0"/>
+</joint>
+<joint name="l_f_h_motor_joint" type="fixed">
+  <origin xyz="-0.105 -0.003 0.153" rpy="0 0 ${pi}" />
   <parent link="l_f_hip"/>
   <child link="l_f_h_motor"/>
   <axis xyz="0 0 1" rpy="0 0 0"/>
-</joint-->
+</joint>
 <joint name="r_f_h_motor_joint"  type="fixed">
-  <origin xyz="-0.010 -0.165 0.088" rpy="0 0 0" />
+  <origin xyz="-0.105 -0.003 0.153" rpy="0 0 -${pi}"/>
   <parent link="r_f_hip"/>
   <child link="r_f_h_motor"/>
@@ -397,5 +397,5 @@
 </joint>
 <joint name="l_b_h_motor_joint"  type="fixed">
-  <origin xyz="-0.016 0.165 0.088" rpy="0 0 0" />
+  <origin xyz="-0.105 0.003 0.153" rpy="0 0 ${pi}" />
   <parent link="l_b_hip"/>
   <child link="l_b_h_motor"/>
@@ -403,35 +403,39 @@
 </joint>
 <joint name="r_b_h_motor_joint"  type="fixed">
-  <origin xyz="-0.010 -0.165 0.088" rpy="0 0 0" />
+  <origin xyz="-0.105 -0.003 0.153" rpy="0 0 ${pi}" />
   <parent link="r_b_hip"/>
   <child link="r_b_h_motor"/>
   <axis xyz="0 0 1" rpy="0 0 0"/>
 </joint>
-<!--joint name="l_f_leg_joint"  type="fixed">
-  <origin xyz="-0.006 0.07 -0.077" rpy="0 0 0" />
+<joint name="l_f_leg_joint"  type="revolute">
+  <origin xyz="0.075 -0.0002 -0.077" rpy="0 0 ${pi}" />
   <parent link="l_f_h_motor"/>
   <child link="l_f_leg"/>
-  <axis xyz="0 0 1" rpy="0 0 0"/>
-</joint-->
-<joint name="l_b_leg_joint"  type="fixed">
-  <origin xyz="-0.006 0.07 -0.077" rpy="0 0 0" />
+  <limit lower="${joint_lower_limit}" upper="${joint_upper_limit}" effort="${joint_effort}" velocity="${joint_velocity}"/>
+  <axis xyz="0 0 1" rpy="0 0 0"/>
+</joint>
+<joint name="l_b_leg_joint"  type="revolute">
+  <origin xyz="0.075 0.0002 -0.077" rpy="0 0 ${pi}" />
   <parent link="l_b_h_motor"/>
   <child link="l_b_leg"/>
-  <axis xyz="0 0 1" rpy="0 0 0"/>
-</joint>
-<joint name="r_f_leg_joint"  type="fixed">
-  <origin xyz="-0.006 -0.07 -0.077" rpy="0 0 0" />
+  <limit lower="${joint_lower_limit}" upper="${joint_upper_limit}" effort="${joint_effort}" velocity="${joint_velocity}"/>
+  <axis xyz="0 0 1" rpy="0 0 0"/>
+</joint>
+<joint name="r_f_leg_joint"  type="revolute">
+  <origin xyz="0.075 -0.0002 -0.077" rpy="0 0 ${pi}" />
   <parent link="r_f_h_motor"/>
   <child link="r_f_leg"/>
-  <axis xyz="0 0 1" rpy="0 0 0"/>
-</joint>
-<joint name="r_b_leg_joint"  type="fixed">
-  <origin xyz="-0.006 -0.07 -0.077" rpy="0 0 0" />
+  <limit lower="${joint_lower_limit}" upper="${joint_upper_limit}" effort="${joint_effort}" velocity="${joint_velocity}"/>
+  <axis xyz="0 0 1" rpy="0 0 0"/>
+</joint>
+<joint name="r_b_leg_joint"  type="revolute">
+  <origin xyz="0.075 0.0002 -0.077" rpy="0 0 ${pi}" />
   <parent link="r_b_h_motor"/>
   <child link="r_b_leg"/>
+  <limit lower="${joint_lower_limit}" upper="${joint_upper_limit}" effort="${joint_effort}" velocity="${joint_velocity}"/>
   <axis xyz="0 0 1" rpy="0 0 0"/>
 </joint>
 <!--######################################################################################################################################-->
-<!--transmission name="l_f_motor_transmission">
+<transmission name="l_f_motor_transmission">
   <type>transmission_interface/SimpleTransmission</type>
   <joint name="l_f_motor_joint">
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