Commit message: adding limit to joint

File: insect_description/urdf/insect.urdf.xacro (robot description, xacro)
@@ -308,6 +308,6 @@
 <!--#########################################################################################################################################-->
 <!-- Joint properties -->
-<xacro:property name="joint_lower_limit" value="-${3.14}"/>
-<xacro:property name="joint_upper_limit" value="${3.14}"/>
+<xacro:property name="joint_lower_limit" value="-${pi/4}"/>
+<xacro:property name="joint_upper_limit" value="${pi/4}"/>
 <xacro:property name="joint_effort" value="6.0"/>
 <xacro:property name="joint_velocity" value="0.524"/>
@@ -360,5 +360,7 @@
   <parent link="l_f_motor"/>
   <child link="l_f_hip"/>
-  <limit lower="${joint_lower_limit}" upper="${joint_upper_limit}" effort="${joint_effort}" velocity="${joint_velocity}"/>
+  <dynamics damping="0.1" friction="0"/>
+  <limit lower="${joint_lower_limit}" upper="${joint_upper_limit}" effort="${joint_effort}" velocity="${joint_velocity}"/>
+  <safety_controller k_position="100" k_velocity="100" soft_lower_limit="-10.5236" soft_upper_limit="10.5236"/>
   <axis xyz="0 0 1"/>
 </joint>
@@ -367,5 +369,7 @@
   <parent link="r_f_motor"/>
   <child link="r_f_hip"/>
-  <limit lower="${joint_lower_limit}" upper="${joint_upper_limit}" effort="${joint_effort}" velocity="${joint_velocity}"/>
+  <dynamics damping="0.1" friction="0"/>
+  <limit lower="${joint_lower_limit}" upper="${joint_upper_limit}" effort="${joint_effort}" velocity="${joint_velocity}"/>
+  <safety_controller k_position="100" k_velocity="100" soft_lower_limit="-10.5236" soft_upper_limit="10.5236"/>
   <axis xyz="0 0 1" rpy="0 0 0"/>
 </joint>
@@ -374,6 +378,8 @@
   <parent link="l_b_motor"/>
   <child link="l_b_hip"/>
-  <axis xyz="0 0 1" rpy="0 0 0"/>
-  <limit lower="${joint_lower_limit}" upper="${joint_upper_limit}" effort="${joint_effort}" velocity="${joint_velocity}"/>
+  <dynamics damping="0.1" friction="0"/>
+  <axis xyz="0 0 1" rpy="0 0 0"/>
+  <limit lower="${joint_lower_limit}" upper="${joint_upper_limit}" effort="${joint_effort}" velocity="${joint_velocity}"/>
+  <safety_controller k_position="100" k_velocity="100" soft_lower_limit="-10.5236" soft_upper_limit="10.5236"/>
 </joint>
  <joint name="r_b_hip_joint"  type="revolute">
@@ -381,5 +387,7 @@
   <parent link="r_b_motor"/>
   <child link="r_b_hip"/>
-  <limit lower="${joint_lower_limit}" upper="${joint_upper_limit}" effort="${joint_effort}" velocity="${joint_velocity}"/>
+  <dynamics damping="0.1" friction="0"/>
+  <limit lower="${joint_lower_limit}" upper="${joint_upper_limit}" effort="${joint_effort}" velocity="${joint_velocity}"/>
+  <safety_controller k_position="100" k_velocity="100" soft_lower_limit="-10.5236" soft_upper_limit="10.5236"/>
   <axis xyz="0 0 1" rpy="0 0 0"/>
 </joint>
@@ -412,6 +420,8 @@
   <parent link="l_f_h_motor"/>
   <child link="l_f_leg"/>
-  <limit lower="${joint_lower_limit}" upper="${joint_upper_limit}" effort="${joint_effort}" velocity="${joint_velocity}"/>
-  <axis xyz="0 0 1" rpy="0 0 0"/>
+  <dynamics damping="0.1" friction="0"/>
+  <limit lower="${joint_lower_limit}" upper="${joint_upper_limit}" effort="${joint_effort}" velocity="${joint_velocity}"/>
+  <safety_controller k_position="100" k_velocity="100" soft_lower_limit="-10.5236" soft_upper_limit="10.5236"/>
+  <axis xyz="0 1 0" rpy="0 0 0"/>
 </joint>
 <joint name="l_b_leg_joint"  type="revolute">
@@ -419,6 +429,8 @@
   <parent link="l_b_h_motor"/>
   <child link="l_b_leg"/>
-  <limit lower="${joint_lower_limit}" upper="${joint_upper_limit}" effort="${joint_effort}" velocity="${joint_velocity}"/>
-  <axis xyz="0 0 1" rpy="0 0 0"/>
+  <dynamics damping="0.1" friction="0"/>
+  <limit lower="${joint_lower_limit}" upper="${joint_upper_limit}" effort="${joint_effort}" velocity="${joint_velocity}"/>
+  <safety_controller k_position="100" k_velocity="100" soft_lower_limit="-10.5236" soft_upper_limit="10.5236"/>
+  <axis xyz="0 1 0" rpy="0 0 0"/>
 </joint>
 <joint name="r_f_leg_joint"  type="revolute">
@@ -426,6 +438,8 @@
   <parent link="r_f_h_motor"/>
   <child link="r_f_leg"/>
-  <limit lower="${joint_lower_limit}" upper="${joint_upper_limit}" effort="${joint_effort}" velocity="${joint_velocity}"/>
-  <axis xyz="0 0 1" rpy="0 0 0"/>
+  <dynamics damping="0.1" friction="0"/>
+  <limit lower="${joint_lower_limit}" upper="${joint_upper_limit}" effort="${joint_effort}" velocity="${joint_velocity}"/>
+  <safety_controller k_position="100" k_velocity="100" soft_lower_limit="-10.5236" soft_upper_limit="10.5236"/>
+  <axis xyz="0 1 0" rpy="0 0 0"/>
 </joint>
 <joint name="r_b_leg_joint"  type="revolute">
@@ -433,6 +447,8 @@
   <parent link="r_b_h_motor"/>
   <child link="r_b_leg"/>
-  <limit lower="${joint_lower_limit}" upper="${joint_upper_limit}" effort="${joint_effort}" velocity="${joint_velocity}"/>
-  <axis xyz="0 0 1" rpy="0 0 0"/>
+  <dynamics damping="0.1" friction="0"/>
+  <limit lower="${joint_lower_limit}" upper="${joint_upper_limit}" effort="${joint_effort}" velocity="${joint_velocity}"/>
+  <safety_controller k_position="100" k_velocity="100" soft_lower_limit="-10.5236" soft_upper_limit="10.5236"/>
+  <axis xyz="0 1 0" rpy="0 0 0"/>
 </joint>
 <!--######################################################################################################################################-->
@@ -467,5 +483,5 @@
     </actuator>
   </transmission>
-  <transmission name="r_b_motor">
+  <transmission name="r_b_motor_transmission">
     <type>transmission_interface/SimpleTransmission</type>
     <joint name="r_b_motor_joint">
