Commit message: kinematics of insect

File: insect_1_description/urdf/insect.urdf (4th copy).xacro (robot description, xacro)
@@ -18,12 +18,12 @@
  </xacro:macro>
  <!--#####################################################################################-->
-<!--link name= "world"/>
+<link name= "world"/>
 <joint name="world_joint" type="fixed">
-  <origin xyz="0.155823674040498 -0.197142204072068 0.168908258984982 " rpy="0 0 0" />
+  <origin xyz="0.225625426875454 -0.0726422157817547  0.05" rpy="0 0 0" />
   <origin xyz="0 0 0" rpy="0 0 0" />
   <parent link="world" />
   <child link="torso_base" />
   <axis xyz="1 0 0" />
-</joint-->
+</joint>
 <!--################################################################################################-->
   <!--IMU sensor_link-->
@@ -101,5 +101,5 @@
    </link>
    <joint name="hokuyo_joint" type="fixed">
-       <origin xyz="0.155 -0.10 0.28" rpy="0 0 ${pi/2  }"/>
+       <origin xyz="0.155 -0.18 0.28" rpy="0 0 ${pi/2  }"/>
        <parent link="torso_base"/>
        <child link="hokuyo_link"/>
@@ -108,18 +108,5 @@
 <!--#######################################################################################################-->
 <link name="torso_base">
-  <inertial>
-    <origin
-      xyz="0.155823674040498 -0.197142204072068 0.168908258984982"
-      rpy="0 0 0" />
-    <mass
-      value="1.09435213027821" />
-    <inertia
-      ixx="1.0"
-      ixy="0"
-      ixz="0"
-      iyy="1.0"
-      iyz="0"
-      izz="1.0" />
-  </inertial>
+  <xacro:default_inertial mass="1.09435213027821"/>
   <visual>
     <origin xyz="0 0 0" rpy="0 0 0" />

File: insect_1_description/urdf/insect2.urdf.xacro (robot description, xacro)
@@ -2,4 +2,10 @@
 <robot name="insect" xmlns:xacro="http://www.ros.org/wiki/xacro">
 <!--###############################################################################-->
+<xacro:property name="hip_len" value="0.148" />
+<xacro:property name="limb_len" value="0.219" />
+<xacro:property name="torso_len" value="0.05" />
+<xacro:property name="torso_width" value="0.05" />
+<xacro:property name="torso_hight" value="0.05" />
+<!--##################################################################################-->
 <!-- Joint properties -->
 <xacro:property name="pi" value="3.1415926535897931"/>

File: insect_robot_3/urdf/insect2.urdf.xacro (robot description, xacro)
@@ -2,4 +2,10 @@
 <robot name="insect" xmlns:xacro="http://www.ros.org/wiki/xacro">
 <!--###############################################################################-->
+<xacro:property name="hip_len" value="0.148" />
+<xacro:property name="limb_len" value="0.219" />
+<xacro:property name="torso_len" value="0.3" />
+<xacro:property name="torso_width" value="0.2" />
+<xacro:property name="torso_hight" value="0.125" />
+<!--##################################################################################-->
 <!-- Joint properties -->
 <xacro:property name="pi" value="3.1415926535897931"/>
@@ -18,5 +24,5 @@
  </xacro:macro>
  <!--#####################################################################################-->
-<!--link name= "world"/>
+<link name= "world"/>
 <joint name="world_joint" type="fixed">
   <origin xyz="0.155823674040498 -0.197142204072068 0.168908258984982 " rpy="0 0 0" />
@@ -25,5 +31,5 @@
   <child link="torso_base" />
   <axis xyz="1 0 0" />
-</joint-->
+</joint>
 <!--################################################################################################-->
   <!--IMU sensor_link-->
